File: FishLight-v01.brd (EAGLE design)
At the start: 85.1 x 85.1 mm, 6 parts, among them U1 ARDUINO_SHIELDARDUINO_SHIELD_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

Commit message: Fishlight_PCB: Updated the schematic and layout
Updated the schematic and layout to add power and ground planes and to
swap out my old parts for my updated library parts.
Parts:
- removed U$1: RTCBREAKOUT, Mikes-Stuff:RTCBREAKOUT
- added FRAME1: FRAME-LETTER, SparkFun-Aesthetics:CREATIVE_COMMONS
- added U2: RTCBREAKOUT, Mikes-Stuff:RTCBREAKOUT
- U1: value ARDUINO_SHIELDARDUINO_SHIELD_FLIPPED -> ARDUINO_SHIELDFLIPPED
Connections:
- net 5V: now also U2.5; no longer U$1.5
- net GND: now also U2.4; no longer U$1.4
- net SCL: now also U2.2; no longer U$1.2
- net SDA: now also U2.1; no longer U$1.1
- net SQW: now also U2.3; no longer U$1.3
Changed lines of the file:
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@@
 <layer number="23" name="tOrigins" color="15" fill="1" visible="yes" active="yes"/>
 <layer number="24" name="bOrigins" color="15" fill="1" visible="yes" active="yes"/>
-<layer number="25" name="tNames" color="7" fill="1" visible="yes" active="yes"/>
-<layer number="26" name="bNames" color="7" fill="1" visible="yes" active="yes"/>
-<layer number="27" name="tValues" color="7" fill="1" visible="yes" active="yes"/>
-<layer number="28" name="bValues" color="7" fill="1" visible="yes" active="yes"/>
+<layer number="25" name="tNames" color="7" fill="1" visible="no" active="yes"/>
+<layer number="26" name="bNames" color="7" fill="1" visible="no" active="yes"/>
+<layer number="27" name="tValues" color="7" fill="1" visible="no" active="yes"/>
+<layer number="28" name="bValues" color="7" fill="1" visible="no" active="yes"/>
 <layer number="29" name="tStop" color="7" fill="3" visible="no" active="yes"/>
 <layer number="30" name="bStop" color="7" fill="6" visible="no" active="yes"/>
@@
 <layer number="37" name="tTest" color="7" fill="1" visible="no" active="yes"/>
 <layer number="38" name="bTest" color="7" fill="1" visible="no" active="yes"/>
-<layer number="39" name="tKeepout" color="4" fill="11" visible="yes" active="yes"/>
-<layer number="40" name="bKeepout" color="1" fill="11" visible="yes" active="yes"/>
+<layer number="39" name="tKeepout" color="4" fill="11" visible="no" active="yes"/>
+<layer number="40" name="bKeepout" color="1" fill="11" visible="no" active="yes"/>
 <layer number="41" name="tRestrict" color="4" fill="10" visible="no" active="yes"/>
 <layer number="42" name="bRestrict" color="1" fill="10" visible="no" active="yes"/>
@@
 <layer number="49" name="Reference" color="7" fill="1" visible="no" active="yes"/>
 <layer number="50" name="dxf" color="7" fill="1" visible="no" active="no"/>
-<layer number="51" name="tDocu" color="13" fill="1" visible="yes" active="yes"/>
-<layer number="52" name="bDocu" color="5" fill="1" visible="yes" active="yes"/>
+<layer number="51" name="tDocu" color="6" fill="1" visible="yes" active="yes"/>
+<layer number="52" name="bDocu" color="5" fill="1" visible="no" active="yes"/>
 <layer number="53" name="tGND_GNDA" color="7" fill="9" visible="no" active="no"/>
 <layer number="54" name="bGND_GNDA" color="1" fill="9" visible="no" active="no"/>
@@
 <wire x1="85.09" y1="85.09" x2="0" y2="85.08" width="0" layer="20"/>
 <wire x1="0" y1="85.08" x2="0" y2="0" width="0" layer="20"/>
+<rectangle x1="1.27" y1="1.27" x2="83.82" y2="83.82" layer="16"/>
+<rectangle x1="1.27" y1="1.27" x2="83.82" y2="83.82" layer="1"/>
 </plain>
 <attributes>
@@
 <element name="STANDOFF3" library="SparkFun-Electromechanical" package="STAND-OFF" value="STAND-OFF" x="82.55" y="2.54"/>
 <element name="STANDOFF4" library="SparkFun-Electromechanical" package="STAND-OFF" value="STAND-OFF" x="2.54" y="2.54"/>
-<element name="U1" library="Mikes-Stuff" package="DUEMILANOVE_SHIELD_NOHOLES" value="ARDUINO_SHIELDARDUINO_SHIELD_FLIPPED" x="6.35" y="85.09" smashed="yes" rot="R180"/>
-<element name="U$1" library="Mikes-Stuff" package="RTCBREAKOUT" value="RTCBREAKOUT" x="36.83" y="24.13" rot="R270"/>
+<element name="FRAME1" library="SparkFun-Aesthetics" package="CREATIVE_COMMONS" value="FRAME-LETTER" x="21.59" y="-8.89"/>
+<element name="U1" library="Mikes-Stuff" package="DUEMILANOVE_SHIELD_NOHOLES" value="ARDUINO_SHIELDFLIPPED" x="6.35" y="85.09" rot="R180"/>
+<element name="U2" library="Mikes-Stuff" package="RTCBREAKOUT" value="RTCBREAKOUT" x="22.86" y="24.13" rot="R270"/>
 </elements>
 <signals>
 <signal name="SDA">
 <contactref element="U1" pad="A4"/>
-<contactref element="U$1" pad="1"/>
-<wire x1="57.15" y1="21.59" x2="57.15" y2="33.02" width="0" layer="19" extent="1-1"/>
+<contactref element="U2" pad="1"/>
+<wire x1="57.15" y1="33.02" x2="43.18" y2="21.59" width="0" layer="19" extent="1-1"/>
 </signal>
 <signal name="SCL">
 <contactref element="U1" pad="A5"/>
-<contactref element="U$1" pad="2"/>
-<wire x1="54.61" y1="21.59" x2="57.15" y2="30.48" width="0" layer="19" extent="1-1"/>
+<contactref element="U2" pad="2"/>
+<wire x1="57.15" y1="30.48" x2="40.64" y2="21.59" width="0" layer="19" extent="1-1"/>
 </signal>
 <signal name="GND">
@@
 <contactref element="U1" pad="GND@1"/>
 <contactref element="U1" pad="GND@0"/>
-<contactref element="U$1" pad="4"/>
+<contactref element="U2" pad="4"/>
+<wire x1="57.15" y1="53.34" x2="35.56" y2="21.59" width="0" layer="19" extent="1-1"/>
 <wire x1="57.15" y1="50.8" x2="57.15" y2="53.34" width="0" layer="19" extent="1-1"/>
 <wire x1="8.89" y1="67.31" x2="57.15" y2="53.34" width="0" layer="19" extent="1-1"/>
-<wire x1="49.53" y1="21.59" x2="8.89" y2="67.31" width="0" layer="19" extent="1-1"/>
 </signal>
 <signal name="5V">
 <contactref element="U1" pad="5V"/>
-<contactref element="U$1" pad="5"/>
-<wire x1="46.99" y1="21.59" x2="57.15" y2="55.88" width="0" layer="19" extent="1-1"/>
+<contactref element="U2" pad="5"/>
+<wire x1="57.15" y1="55.88" x2="33.02" y2="21.59" width="0" layer="19" extent="1-1"/>
 </signal>
 <signal name="SQW">
-<contactref element="U$1" pad="3"/>
+<contactref element="U2" pad="3"/>
 </signal>
 </signals>

Commit message: FishLight_PCB: Added screw terminals
The screw terminals are under M02 and M03 for 2 and 3 pin terminals
respectfully.  These will be used to connect things like power and
ground cables to my LED strings.  I may need to get less than I
currently put in.  Though it might be nice to totally breakout every
Arduino pin to a header.
Parts:
- added JP1, JP2, JP3, JP4, JP5, JP6, JP7, JP8: (no value), SparkFun-Connectors:SCREWTERMINAL-3.5MM-3_LOCK.007S
- added JP9: M023.5MM, SparkFun-Connectors:SCREWTERMINAL-3.5MM-2
- moved U2 7.73 mm to (30.5, 22.9)
- moved U1 5.24 mm to (11.4, 83.8)
Changed lines of the file:
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@@
 <layer number="106" name="bPlate" color="7" fill="1" visible="no" active="yes"/>
 <layer number="107" name="Crop" color="7" fill="1" visible="no" active="yes"/>
+<layer number="108" name="tplace-old" color="10" fill="1" visible="yes" active="yes"/>
+<layer number="109" name="ref-old" color="11" fill="1" visible="yes" active="yes"/>
 <layer number="116" name="Patch_BOT" color="9" fill="4" visible="no" active="yes"/>
 <layer number="121" name="_tsilk" color="7" fill="1" visible="no" active="yes"/>
@@
 <element name="STANDOFF4" library="SparkFun-Electromechanical" package="STAND-OFF" value="STAND-OFF" x="2.54" y="2.54"/>
 <element name="FRAME1" library="SparkFun-Aesthetics" package="CREATIVE_COMMONS" value="FRAME-LETTER" x="21.59" y="-8.89"/>
-<element name="U1" library="Mikes-Stuff" package="DUEMILANOVE_SHIELD_NOHOLES" value="ARDUINO_SHIELDFLIPPED" x="6.35" y="85.09" rot="R180"/>
-<element name="U2" library="Mikes-Stuff" package="RTCBREAKOUT" value="RTCBREAKOUT" x="22.86" y="24.13" rot="R270"/>
+<element name="U1" library="Mikes-Stuff" package="DUEMILANOVE_SHIELD_NOHOLES" value="ARDUINO_SHIELDFLIPPED" x="11.43" y="83.82" rot="R180"/>
+<element name="U2" library="Mikes-Stuff" package="RTCBREAKOUT" value="RTCBREAKOUT" x="30.48" y="22.86" rot="R270"/>
+<element name="JP1" library="SparkFun-Connectors" package="SCREWTERMINAL-3.5MM-3_LOCK.007S" value="" x="80.01" y="7.62" rot="R90"/>
+<element name="JP2" library="SparkFun-Connectors" package="SCREWTERMINAL-3.5MM-3_LOCK.007S" value="" x="5.08" y="24.13" rot="R270"/>
+<element name="JP3" library="SparkFun-Connectors" package="SCREWTERMINAL-3.5MM-3_LOCK.007S" value="" x="5.08" y="35.56" rot="R270"/>
+<element name="JP4" library="SparkFun-Connectors" package="SCREWTERMINAL-3.5MM-3_LOCK.007S" value="" x="5.08" y="46.99" rot="R270"/>
+<element name="JP5" library="SparkFun-Connectors" package="SCREWTERMINAL-3.5MM-3_LOCK.007S" value="" x="80.01" y="53.34" rot="R90"/>
+<element name="JP6" library="SparkFun-Connectors" package="SCREWTERMINAL-3.5MM-3_LOCK.007S" value="" x="80.01" y="41.91" rot="R90"/>
+<element name="JP7" library="SparkFun-Connectors" package="SCREWTERMINAL-3.5MM-3_LOCK.007S" value="" x="80.01" y="30.48" rot="R90"/>
+<element name="JP8" library="SparkFun-Connectors" package="SCREWTERMINAL-3.5MM-3_LOCK.007S" value="" x="80.01" y="19.05" rot="R90"/>
+<element name="JP9" library="SparkFun-Connectors" package="SCREWTERMINAL-3.5MM-2" value="M023.5MM" x="5.08" y="13.081" rot="R270"/>
 </elements>
 <signals>
@@
 <contactref element="U1" pad="A4"/>
 <contactref element="U2" pad="1"/>
-<wire x1="57.15" y1="33.02" x2="43.18" y2="21.59" width="0" layer="19" extent="1-1"/>
+<wire x1="62.23" y1="31.75" x2="50.8" y2="20.32" width="0" layer="19" extent="1-1"/>
 </signal>
 <signal name="SCL">
 <contactref element="U1" pad="A5"/>
 <contactref element="U2" pad="2"/>
-<wire x1="57.15" y1="30.48" x2="40.64" y2="21.59" width="0" layer="19" extent="1-1"/>
+<wire x1="62.23" y1="29.21" x2="48.26" y2="20.32" width="0" layer="19" extent="1-1"/>
 </signal>
 <signal name="GND">
@@
 <contactref element="U1" pad="GND@0"/>
 <contactref element="U2" pad="4"/>
-<wire x1="57.15" y1="53.34" x2="35.56" y2="21.59" width="0" layer="19" extent="1-1"/>
-<wire x1="57.15" y1="50.8" x2="57.15" y2="53.34" width="0" layer="19" extent="1-1"/>
-<wire x1="8.89" y1="67.31" x2="57.15" y2="53.34" width="0" layer="19" extent="1-1"/>
+<wire x1="62.23" y1="52.07" x2="43.18" y2="20.32" width="0" layer="19" extent="1-1"/>
+<wire x1="62.23" y1="49.53" x2="62.23" y2="52.07" width="0" layer="19" extent="1-1"/>
+<wire x1="13.97" y1="66.04" x2="62.23" y2="52.07" width="0" layer="19" extent="1-1"/>
 </signal>
 <signal name="5V">
 <contactref element="U1" pad="5V"/>
 <contactref element="U2" pad="5"/>
-<wire x1="57.15" y1="55.88" x2="33.02" y2="21.59" width="0" layer="19" extent="1-1"/>
+<wire x1="62.23" y1="54.61" x2="40.64" y2="20.32" width="0" layer="19" extent="1-1"/>
 </signal>
 <signal name="SQW">

Commit message: FishLight_PCB: Connected screw terminals
Connected the screw terminals to the Arduino so that each Arduino pin
has a terminal.  Rearranged the schematic a bit to be more organized and
also added LED screw terminals.
Parts:
- added JP10, JP11, JP12: (no value), SparkFun-Connectors:SCREWTERMINAL-3.5MM-3
- JP1, JP2, JP3, JP4, JP5, JP6, JP7, JP8: device SparkFun-Connectors:SCREWTERMINAL-3.5MM-3_LOCK.007S -> SparkFun-Connectors:SCREWTERMINAL-3.5MM-3
- JP9: value M023.5MM -> (none); device SparkFun-Connectors:SCREWTERMINAL-3.5MM-2 -> SparkFun-Connectors:SCREWTERMINAL-3.5MM-3
- moved JP9 88.0 mm to (81.3, 57.1), turned to 90 degrees
- moved JP1 79.6 mm to (3.81, 30.5), turned to 270 degrees
- moved JP5 79.6 mm to (3.81, 76.2), turned to 270 degrees
- moved FRAME1 37.4 mm to (58.4, -2.54)
- moved JP3 17.8 mm to (3.81, 53.3)
- moved JP2 17.8 mm to (3.81, 41.9)
- moved JP4 17.8 mm to (3.81, 64.8)
- moved JP6 4.02 mm to (81.3, 45.7)
- moved JP7 4.02 mm to (81.3, 34.3)
- moved JP8 4.02 mm to (81.3, 22.9)
- moved U1 3.81 mm to (15.2, 83.8)
Connections:
- new net 3.3V: JP11.1, JP6.1, U1.3.3V
- new net A0: JP7.3, U1.A0
- new net A1: JP7.2, U1.A1
- new net A2: JP7.1, U1.A2
- new net A3: JP8.3, U1.A3
- new net AREF: JP9.3, U1.AREF
- new net D10: JP4.2, U1.D10
- new net D11: JP4.1, U1.D11
- new net D12: JP5.3, U1.D12
- new net D13: JP5.2, U1.D13
- new net D2: JP1.1, U1.D2
- new net D3: JP2.3, U1.D3
- new net D4: JP2.2, U1.D4
- new net D5: JP2.1, U1.D5
- new net D6: JP3.3, U1.D6
- new net D7: JP3.2, U1.D7
- new net D8: JP3.1, U1.D8
- new net D9: JP4.3, U1.D9
- new net LED1: JP10.1
- new net LED2: JP10.2
- new net LED3: JP10.3
- new net RES: JP9.2, U1.RES
- new net RX: JP1.2, U1.RX
- new net TX: JP1.3, U1.TX
- new net VIN: JP9.1, U1.VIN
- net 5V: now also JP11.3, JP6.3
- net GND: now also JP11.2, JP12.1, JP12.2, JP12.3, JP5.1, JP6.2
- net SCL: now also JP8.1
- net SDA: now also JP8.2
Other:
- board text added: "3.3V"
- board text added: "5V"
- board text added: "A0"
- board text added: "A1"
- board text added: "A2"
- board text added: "A3"
- board text added: "A4"
- board text added: "A5"
- board text added: "Aref"
- board text added: "BL"
- board text added: "CW"
- board text added: "CW LED"
- board text added: "D0"
- board text added: "D1"
- board text added: "D10*"
- board text added: "D11*"
- board text added: "D12"
- board text added: "D13"
- board text added: "D2"
- board text added: "D3*"
- board text added: "D4"
- board text added: "D5*"
- board text added: "D6*"
- board text added: "D7"
- board text added: "D8"
- board text added: "D9*"
- board text added: "GND"
- board text added: "LED GND"
- board text added: "Rst"
- board text added: "Vin"
- board text added: "WW"

Commit message: FishLight_PCB: Added CAT4101
Created a symbol and layout for the CAT4101 device.  Hooked up the power
and ground pins with a bypass cap and connected the PWM pins.  Also
added pull ups for the I2C bus.
Parts:
- added U$1, U$2, U$3, U$4, U$5, U$6: CAT4101CAT4101, Mikes-Stuff:TO-263
Changed lines of the file:
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@@
 <element name="JP11" library="SparkFun-Connectors" package="SCREWTERMINAL-3.5MM-3" value="" x="15.24" y="3.81"/>
 <element name="JP12" library="SparkFun-Connectors" package="SCREWTERMINAL-3.5MM-3" value="" x="81.28" y="8.89" rot="R90"/>
+<element name="U$1" library="Mikes-Stuff" package="TO-263" value="CAT4101CAT4101" x="-6.35" y="0"/>
+<element name="U$2" library="Mikes-Stuff" package="TO-263" value="CAT4101CAT4101" x="-17.78" y="0"/>
+<element name="U$3" library="Mikes-Stuff" package="TO-263" value="CAT4101CAT4101" x="-29.21" y="0"/>
+<element name="U$4" library="Mikes-Stuff" package="TO-263" value="CAT4101CAT4101" x="-40.64" y="0"/>
+<element name="U$5" library="Mikes-Stuff" package="TO-263" value="CAT4101CAT4101" x="-52.07" y="0"/>
+<element name="U$6" library="Mikes-Stuff" package="TO-263" value="CAT4101CAT4101" x="-63.5" y="0"/>
 </elements>
 <signals>

Commit message: FishLight_PCB: Added AD5246 Digital Pot
Added the AD5246 Digital Potentiometer.  This is a 5Kohm Digital
Potentiometer with an I2C interface and a range of approximately 100ohm
- 5100ohm.  This will give me sufficient range to sweep all the way from
100mA to 1000mA on the CAT4101 with a resistance range of about 4990ohm
- 549ohm respectively.
Parts:
- added C1, C10, C11, C12, C2, C3, C4, C5, C6, C7, C8, C9: 0.1uF, SparkFun-Capacitors:0603-CAP
- added R1, R2: (no value), SparkFun-Resistors:0603-RES
- added U10, U11, U12, U13, U14, U9: AD5246TSSOT6, Mikes-Stuff:TSSOT6
- U3, U4, U5, U6, U7, U8: value CAT4101CAT4101 -> CAT4101TO-263
- renumbered U$1 to U3, U$2 to U4, U$3 to U5, U$4 to U6, U$5 to U7, U$6 to U8
Connections:
- new net LG1: JP12.3, U3.5
- new net LG2: JP12.2, U4.5
- new net LG3: JP12.1, U5.5
- new net LR1: U3.4, U9.5
- new net LR2: U10.5, U4.4
- new net LR3: U11.5, U5.4
- new net N$1: U14.4
- new net N$10: U9.4
- new net N$13: U6.1
- new net N$14: U6.4
- new net N$15: U6.5
- new net N$16: U7.1
- new net N$17: U7.4
- new net N$18: U7.5
- new net N$19: U8.1
- new net N$2: U13.4
- new net N$20: U8.4
- new net N$21: U8.5
- new net N$23: U10.4
- new net N$27: U11.4
- new net N$3: U12.4
- net 5V: now also C1.1, C10.1, C11.1, C12.1, C2.1, C3.1, C4.1, C5.1, C6.1, C7.1, C8.1, C9.1, R1.2, R2.2, U10.1, U11.1, U12.1, U13.1, U14.1, U3.2, U4.2, U5.2, U6.2, U7.2, U8.2, U9.1
- net D10: now also U4.1
- net D11: now also U5.1
- net D9: now also U3.1
- net GND: now also C1.2, C10.2, C11.2, C12.2, C2.2, C3.2, C4.2, C5.2, C6.2, C7.2, C8.2, C9.2, U10.2, U10.6, U11.2, U11.6, U12.2, U12.6, U13.2, U13.6, U14.2, U14.6, U3.3, U3.6, U4.3, U4.6, U5.3, U5.6, U6.3, U6.6, U7.3, U7.6, U8.3, U8.6, U9.2, U9.6; no longer JP12.1, JP12.2, JP12.3
- net SCL: now also R2.1, U10.3, U11.3, U12.3, U13.3, U14.3, U9.3
- net SDA: now also R1.1

Commit message: FishLight_PCB: Added CD74HC4067 16x MUX
Added the CD74HC4067 16-Channel MUX.  This is going to control which
digital pot gets written to since they all have the same I2C address.  I
hope it will be fast enough to write a single register on each pot.
Pulled the SSOP20 package from Sparkfun and modified it for a 24 pin
package.  Hooked up the SDA signals on 3 of the pots and the Arduino.
Still need to connect the Digital control signals S0-3.  Need to choose
which pins those will be.
Parts:
- added C13: 0.1uF, SparkFun-Capacitors:0603-CAP
- added U$1: CD74HC4067SSOP24, Mikes-Stuff:SSOP24
Connections:
- removed net N$10: U9.4
- removed net N$23: U10.4
- removed net N$27: U11.4
- new net N$11: U$1.10
- new net N$12: U$1.11
- new net N$24: U$1.13
- new net N$25: U$1.14
- new net N$28: U$1.15
- new net N$7: U$1.6
- new net N$8: U$1.5
- new net N$9: U$1.4
- new net SDA1: U$1.9, U9.4
- new net SDA2: U$1.8, U10.4
- new net SDA3: U$1.7, U11.4
- net 5V: now also C13.2, U$1.24
- net GND: now also C13.1, U$1.12
- net SDA: now also U$1.1
Changed lines of the file:
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@@
 <attribute name="PROD_ID" value="CAP-08604" x="-67.31" y="-97.79" size="1.27" layer="27" ratio="15" display="off"/>
+</element>
+<element name="U$1" library="Mikes-Stuff" package="SSOP24" value="CD74HC4067SSOP24" x="-64.77" y="-104.14"/>
+<element name="C13" library="SparkFun-Capacitors" package="0603-CAP" value="0.1uF" x="-67.31" y="-110.49">
+<attribute name="PROD_ID" value="CAP-00810" x="-67.31" y="-110.49" size="1.27" layer="27" ratio="15" display="off"/>
 </element>
 </elements>
@@
 <contactref element="JP8" pad="2"/>
 <contactref element="R1" pad="1"/>
-<wire x1="66.04" y1="31.75" x2="81.28" y2="26.36" width="0" layer="19" extent="1-1"/>
-<wire x1="50.8" y1="20.32" x2="66.04" y2="31.75" width="0" layer="19" extent="1-1"/>
-<wire x1="-68.16" y1="-27.94" x2="50.8" y2="20.32" width="0" layer="19" extent="1-1"/>
+<contactref element="U$1" pad="1"/>
+<wire x1="-68.16" y1="-27.94" x2="-67.695" y2="-107.765" width="0" layer="19" extent="1-1"/>
+<wire x1="50.8" y1="20.32" x2="-68.16" y2="-27.94" width="0" layer="19" extent="1-1"/>
+<wire x1="66.04" y1="31.75" x2="50.8" y2="20.32" width="0" layer="19" extent="1-1"/>
+<wire x1="81.28" y1="26.36" x2="66.04" y2="31.75" width="0" layer="19" extent="1-1"/>
 </signal>
 <signal name="SCL">
@@
 <contactref element="U14" pad="2"/>
 <contactref element="U14" pad="6"/>
+<contactref element="U$1" pad="12"/>
+<contactref element="C13" pad="1"/>
+<wire x1="-62.495" y1="-100.515" x2="-68.16" y2="-110.49" width="0" layer="19" extent="1-1"/>
+<wire x1="-66.46" y1="-97.79" x2="-62.495" y2="-100.515" width="0" layer="19" extent="1-1"/>
 <wire x1="-66.46" y1="-93.98" x2="-66.46" y2="-97.79" width="0" layer="19" extent="1-1"/>
 <wire x1="-66.46" y1="-90.17" x2="-66.46" y2="-93.98" width="0" layer="19" extent="1-1"/>
@@
 <contactref element="U13" pad="1"/>
 <contactref element="U14" pad="1"/>
+<contactref element="U$1" pad="24"/>
+<contactref element="C13" pad="2"/>
+<wire x1="-61.225" y1="-100.515" x2="-66.46" y2="-110.49" width="0" layer="19" extent="1-1"/>
+<wire x1="-68.16" y1="-97.79" x2="-61.225" y2="-100.515" width="0" layer="19" extent="1-1"/>
 <wire x1="-68.16" y1="-93.98" x2="-68.16" y2="-97.79" width="0" layer="19" extent="1-1"/>
 <wire x1="-68.16" y1="-90.17" x2="-68.16" y2="-93.98" width="0" layer="19" extent="1-1"/>
@@
 <wire x1="-27.51" y1="2.1" x2="-67.31" y2="-49.85" width="0" layer="19" extent="1-1"/>
 </signal>
-<signal name="N$10">
-<contactref element="U9" pad="4"/>
-</signal>
-<signal name="N$23">
-<contactref element="U10" pad="4"/>
-</signal>
-<signal name="N$27">
-<contactref element="U11" pad="4"/>
-</signal>
 <signal name="N$1">
 <contactref element="U14" pad="4"/>
@@
 <contactref element="U12" pad="4"/>
 </signal>
+<signal name="SDA1">
+<contactref element="U$1" pad="9"/>
+<contactref element="U9" pad="4"/>
+<wire x1="-66.66" y1="-34.61" x2="-62.495" y2="-107.765" width="0" layer="19" extent="1-1"/>
+</signal>
+<signal name="SDA2">
+<contactref element="U$1" pad="8"/>
+<contactref element="U10" pad="4"/>
+<wire x1="-66.66" y1="-42.23" x2="-63.145" y2="-107.765" width="0" layer="19" extent="1-1"/>
+</signal>
+<signal name="SDA3">
+<contactref element="U$1" pad="7"/>
+<contactref element="U11" pad="4"/>
+<wire x1="-66.66" y1="-49.85" x2="-63.795" y2="-107.765" width="0" layer="19" extent="1-1"/>
+</signal>
+<signal name="N$7">
+<contactref element="U$1" pad="6"/>
+</signal>
+<signal name="N$8">
+<contactref element="U$1" pad="5"/>
+</signal>
+<signal name="N$9">
+<contactref element="U$1" pad="4"/>
+</signal>
+<signal name="N$11">
+<contactref element="U$1" pad="10"/>
+</signal>
+<signal name="N$12">
+<contactref element="U$1" pad="11"/>
+</signal>
+<signal name="N$24">
+<contactref element="U$1" pad="13"/>
+</signal>
+<signal name="N$25">
+<contactref element="U$1" pad="14"/>
+</signal>
+<signal name="N$28">
+<contactref element="U$1" pad="15"/>
+</signal>
 </signals>

Commit message: FishLight_PCB: Added 12V regulator
Added the UA7812 12V regulator.  This will convert my 24V power supply
to 12V to power the Arduino.  This may also power a fan.
Parts:
- removed U14: AD5246TSSOT6, Mikes-Stuff:TSSOT6
- removed U8: CAT4101TO-263, Mikes-Stuff:TO-263
- added JP13, JP14: (no value), SparkFun-Connectors:SCREWTERMINAL-3.5MM-3
- added U$2: UA7812, Mikes-Stuff:D2PAK-3
- C12: value 0.1uF -> 0.33uF
- R1, R2: value (none) -> 10K
- moved C6 106.0 mm to (-78.7, -129.5)
- moved C12 37.4 mm to (-78.7, -133.3)
Connections:
- removed net N$1: U14.4
- removed net N$13: U6.1
- removed net N$14: U6.4
- removed net N$15: U6.5
- removed net N$16: U7.1
- removed net N$17: U7.4
- removed net N$18: U7.5
- removed net N$19: U8.1
- removed net N$2: U13.4
- removed net N$20: U8.4
- removed net N$21: U8.5
- removed net N$7: U$1.6
- removed net N$8: U$1.5
- removed net VIN: JP9.1, U1.VIN
- new net 12V: C6.1, JP9.1, U$2.3, U1.VIN
- new net 24V: C12.1, U$2.1
- new net LED4: JP14.1
- new net LED5: JP14.2
- new net LG4: JP13.3, U6.5
- new net LG5: JP13.2, U7.5
- new net LR4: U12.5, U6.4
- new net LR5: U13.5, U7.4
- new net N$6: JP13.1
- new net SDA4: U$1.6, U12.4
- new net SDA5: U$1.5, U13.4
- net 5V: no longer C12.1, C6.1, U14.1, U8.2
- net D3: now also U6.1
- net D5: now also U7.1
- net GND: now also U$2.2; no longer U14.2, U14.6, U8.3, U8.6
- net N$3: now also JP14.3; no longer U12.4
- net SCL: no longer U14.3
