File: FishLight-v01.brd (EAGLE design)
At the start: 85.1 x 85.1 mm, 48 parts, among them U1 ARDUINO_SHIELDFLIPPED, U10 AD5246TSSOT6, U11 AD5246TSSOT6, U12 AD5246TSSOT6, U13 AD5246TSSOT6, U2 RTCBREAKOUT, U3 CAT4101TO-263, U4 CAT4101TO-263, U5 CAT4101TO-263, U6 CAT4101TO-263, U7 CAT4101TO-263, U9 AD5246TSSOT6

Commit message: FishLight_PCB: Added 5V regulator and 3 pin Molex
Added the L7805 5V regulator.  This may not be necessary unless I want
to use the Spark Core.  The Spark has a max input voltage of 6V, making
the 12V regulator unnecessary.  Perhaps I will pick a regulator that can
be changed to 5V or 12V depending on what I want to use just by changing
one set resistor.  Also added a few 3 pin Molex connectors that I can
use for temperature sensors.  I haven't picked a part for that yet but I
may go with the DS18B20 even tho it is kind of expensive.  But it is
really nice since it has an Arduino library already and it only uses 1
wire to talk to the Arduino and it can have a large number of sensors on
the same wire since they all have different pre-programmed addresses.
Parts:
- added C14: 0.33uF, SparkFun-Capacitors:0603-CAP
- added C15: 0.1uF, SparkFun-Capacitors:0603-CAP
- added JP15, JP16, JP17: (no value), Mikes-Stuff:SCREWTERMINAL-3.5MM-3
- added U15: L7805D2PAK-2, Mikes-Stuff:D2PAK-2
- JP1, JP2, JP3: device SparkFun-Connectors:SCREWTERMINAL-3.5MM-3 -> Mikes-Stuff:MOLEX-1X3
- JP10, JP11, JP12, JP13, JP14, JP4, JP5, JP6, JP7, JP8, JP9: device SparkFun-Connectors:SCREWTERMINAL-3.5MM-3 -> Mikes-Stuff:SCREWTERMINAL-3.5MM-3
- U14: value UA7812 -> UA7812D2PAK-3
- moved JP9 298.5 mm to (-77.5, -195.6), turned to 0 degrees
- moved JP12 277.3 mm to (-77.5, -218.4), turned to 0 degrees
- moved JP6 270.0 mm to (-77.5, -172.7), turned to 0 degrees
- moved JP7 267.0 mm to (-77.5, -180.3), turned to 0 degrees
- moved JP8 263.9 mm to (-77.5, -188.0), turned to 0 degrees
- moved JP5 254.6 mm to (-77.5, -165.1), turned to 0 degrees
- moved JP4 236.6 mm to (-77.5, -157.5), turned to 0 degrees
- moved JP11 233.8 mm to (-77.5, -210.8)
- moved JP10 233.1 mm to (-77.5, -203.2), turned to 0 degrees
- moved JP3 220.5 mm to (-78.7, -151.1), turned to 0 degrees
- moved JP2 204.1 mm to (-78.7, -144.8), turned to 0 degrees
- moved JP1 188.0 mm to (-78.7, -138.4), turned to 0 degrees
- moved JP14 110.0 mm to (-77.5, -233.7)
- moved JP13 110.0 mm to (-77.5, -226.1)
- renumbered U$1 to U8, U$2 to U14
Connections:
- new net N$13: JP1.2
- new net N$2: JP3.2
- new net N$7: JP2.2
- net 12V: now also JP15.1; no longer JP9.1
- net 24V: now also C14.1, U15.1
- net 3.3V: now also JP13.1, JP14.1; no longer JP11.1, JP6.1
- net 5V: now also C15.1, JP1.3, JP13.3, JP14.3, JP2.3, JP3.3, U15.3; no longer JP11.3, JP6.3
- net A0: now also JP17.3; no longer JP7.3
- net A1: now also JP17.2; no longer JP7.2
- net A2: now also JP17.1; no longer JP7.1
- net A3: now also JP16.3; no longer JP8.3
- net AREF: now also JP15.3; no longer JP9.3
- net D10: now also JP7.2; no longer JP4.2
- net D11: now also JP7.1; no longer JP4.1
- net D12: now also JP8.3; no longer JP5.3
- net D13: now also JP8.2; no longer JP5.2
- net D2: now also JP4.1; no longer JP1.1
- net D3: now also JP5.3; no longer JP2.3
- net D4: now also JP5.2; no longer JP2.2
- net D5: now also JP5.1; no longer JP2.1
- net D6: now also JP6.3; no longer JP3.3
- net D7: now also JP6.2; no longer JP3.2
- net D8: now also JP6.1; no longer JP3.1
- net D9: now also JP7.3; no longer JP4.3
- net GND: now also C14.2, C15.2, JP1.1, JP13.2, JP14.2, JP2.1, JP3.1, JP8.1, U15.2; no longer JP11.2, JP5.1, JP6.2
- net LED1: now also JP12.1; no longer JP10.1
- net LED2: now also JP12.2; no longer JP10.2
- net LED3: now also JP12.3; no longer JP10.3
- net LED4: now also JP11.1; no longer JP14.1
- net LED5: now also JP11.2; no longer JP14.2
- net LG1: now also JP9.3; no longer JP12.3
- net LG2: now also JP9.2; no longer JP12.2
- net LG3: now also JP9.1; no longer JP12.1
- net LG4: now also JP10.3; no longer JP13.3
- net LG5: now also JP10.2; no longer JP13.2
- net N$3: now also JP11.3; no longer JP14.3
- net N$6: now also JP10.1; no longer JP13.1
- net RES: now also JP15.2; no longer JP9.2
- net RX: now also JP4.2; no longer JP1.2
- net SCL: now also JP16.1; no longer JP8.1
- net SDA: now also JP16.2; no longer JP8.2
- net TX: now also JP4.3; no longer JP1.3
