File: FishLight-v01.brd (EAGLE design)
At the start: 85.1 x 85.1 mm, 54 parts, among them U1 ARDUINO_SHIELDFLIPPED, U10 AD5246TSSOT6, U11 AD5246TSSOT6, U12 AD5246TSSOT6, U13 AD5246TSSOT6, U14 UA7812D2PAK-3, U15 L7805D2PAK-2, U2 RTCBREAKOUT, U3 CAT4101TO-263, U4 CAT4101TO-263, U5 CAT4101TO-263, U6 CAT4101TO-263, U7 CAT4101TO-263, U8 CD74HC4067SSOP24, U9 AD5246TSSOT6

Commit message: FishLight_PCB: Upgrade to Spark Core
I am planning on using the Spark Core for this project so that I can
have a wireless connection to program the board and get updates on
things like temperature wirelessly.  Added the Spark Core parts library,
the Adafruit parts library, updated a few of my parts and changed to the
Spark Core.
Parts:
- removed U1: ARDUINO_SHIELDFLIPPED, Mikes-Stuff:DUEMILANOVE_SHIELD_NOHOLES
- added U$1: SPARK_CORECORE, Spark:SPARK_CORE
- moved FRAME1 58.5 mm to (0.00, 0.00)
- moved U2 24.2 mm to (29.2, 47.0), turned to 180 degrees
Connections:
- new net A6: U$1.6
- new net A7: U$1.5
- new net D0: U$1.13
- new net D1: U$1.14
- new net RAW: U$1.1
- new net VDDA: U$1.22
- net 12V: no longer U1.VIN
- net 3.3V: no longer U1.3.3V
- net 5V: now also U$1.24; no longer U1.5V
- net A0: now also U$1.12; no longer U1.A0
- net A1: now also U$1.11; no longer U1.A1
- net A2: now also U$1.10; no longer U1.A2
- net A3: now also U$1.9; no longer U1.A3
- net AREF: no longer U1.AREF
- net D10: no longer U1.D10
- net D11: no longer U1.D11
- net D12: no longer U1.D12
- net D13: no longer U1.D13
- net D2: now also U$1.15; no longer U1.D2
- net D3: now also U$1.16; no longer U1.D3
- net D4: now also U$1.17; no longer U1.D4
- net D5: now also U$1.18; no longer U1.D5
- net D6: now also U$1.19; no longer U1.D6
- net D7: now also U$1.20; no longer U1.D7
- net D8: no longer U1.D8
- net D9: no longer U1.D9
- net GND: now also U$1.2, U$1.21; no longer U1.GND@0, U1.GND@1, U1.GND@2
- net RES: now also U$1.23; no longer U1.RES
- net RX: now also U$1.4; no longer U1.RX
- net SCL: now also U$1.8; no longer U1.A5
- net SDA: now also U$1.7; no longer U1.A4
- net TX: now also U$1.3; no longer U1.TX
Other:
- board text removed: "CW LED"

Commit message: FishLight_PCB: Some minor edits
Added pull up resistors on the external temperature sensor headers.
Changed some text.
Parts:
- added R3, R4, R5: 4.7K, SparkFun-Resistors:0603-RES
Connections:
- net 5V: now also R3.2, R4.2, R5.2
- net N$13: now also R5.1
- net N$2: now also R3.1
- net N$7: now also R4.1
Changed lines of the file:
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@@
 </element>
 <element name="U$1" library="Spark" package="SPARK_CORE" value="SPARK_CORECORE" x="53.34" y="48.26"/>
+<element name="R3" library="SparkFun-Resistors" package="0603-RES" value="4.7K" x="-90.17" y="-269.24"/>
+<element name="R4" library="SparkFun-Resistors" package="0603-RES" value="4.7K" x="-90.17" y="-271.78"/>
+<element name="R5" library="SparkFun-Resistors" package="0603-RES" value="4.7K" x="-90.17" y="-274.32"/>
 </elements>
 <signals>
@@
 <contactref element="JP1" pad="3"/>
 <contactref element="U$1" pad="24"/>
+<contactref element="R3" pad="2"/>
+<contactref element="R4" pad="2"/>
+<contactref element="R5" pad="2"/>
 <wire x1="-73.66" y1="-144.78" x2="-73.66" y2="-151.13" width="0" layer="19" extent="1-1"/>
 <wire x1="-73.66" y1="-138.43" x2="-73.66" y2="-144.78" width="0" layer="19" extent="1-1"/>
@@
 <wire x1="-68.16" y1="-8.89" x2="-68.16" y2="-12.7" width="0" layer="19" extent="1-1"/>
 <wire x1="-68.16" y1="-5.08" x2="-68.16" y2="-8.89" width="0" layer="19" extent="1-1"/>
-<wire x1="-53.77" y1="-9.33" x2="-68.16" y2="-5.08" width="0" layer="19" extent="1-1"/>
+<wire x1="-53.77" y1="-9.33" x2="-68.16" y2="-8.89" width="0" layer="19" extent="1-1"/>
 <wire x1="-42.34" y1="-9.33" x2="-53.77" y2="-9.33" width="0" layer="19" extent="1-1"/>
 <wire x1="-30.91" y1="-9.33" x2="-42.34" y2="-9.33" width="0" layer="19" extent="1-1"/>
@@
 <wire x1="-8.05" y1="-9.33" x2="-19.48" y2="-9.33" width="0" layer="19" extent="1-1"/>
 <wire x1="36.83" y1="49.53" x2="-8.05" y2="-9.33" width="0" layer="19" extent="1-1"/>
+<wire x1="62.23" y1="62.23" x2="36.83" y2="49.53" width="0" layer="19" extent="1-1"/>
 <wire x1="-70.47" y1="-226.06" x2="-73.66" y2="-151.13" width="0" layer="19" extent="1-1"/>
 <wire x1="-70.47" y1="-233.68" x2="-70.47" y2="-226.06" width="0" layer="19" extent="1-1"/>
-<wire x1="62.23" y1="62.23" x2="-70.47" y2="-233.68" width="0" layer="19" extent="1-1"/>
-<wire x1="-82.96" y1="-254.44" x2="62.23" y2="62.23" width="0" layer="19" extent="1-1"/>
+<wire x1="-82.96" y1="-254.44" x2="-70.47" y2="-233.68" width="0" layer="19" extent="1-1"/>
 <wire x1="-91.02" y1="-265.43" x2="-82.96" y2="-254.44" width="0" layer="19" extent="1-1"/>
+<wire x1="-89.32" y1="-269.24" x2="-91.02" y2="-265.43" width="0" layer="19" extent="1-1"/>
+<wire x1="-89.32" y1="-271.78" x2="-89.32" y2="-269.24" width="0" layer="19" extent="1-1"/>
+<wire x1="-89.32" y1="-274.32" x2="-89.32" y2="-271.78" width="0" layer="19" extent="1-1"/>
 </signal>
 <signal name="SQW">
@@
 <signal name="N$2">
 <contactref element="JP3" pad="2"/>
+<contactref element="R3" pad="1"/>
+<wire x1="-91.02" y1="-269.24" x2="-76.2" y2="-151.13" width="0" layer="19" extent="1-1"/>
 </signal>
 <signal name="N$7">
 <contactref element="JP2" pad="2"/>
+<contactref element="R4" pad="1"/>
+<wire x1="-91.02" y1="-271.78" x2="-76.2" y2="-144.78" width="0" layer="19" extent="1-1"/>
 </signal>
 <signal name="N$13">
 <contactref element="JP1" pad="2"/>
+<contactref element="R5" pad="1"/>
+<wire x1="-91.02" y1="-274.32" x2="-76.2" y2="-138.43" width="0" layer="19" extent="1-1"/>
 </signal>
 <signal name="RAW">

Commit message: FishLight_PCB: Added 2 digital pots and I-sense R
Added the AD5254 and the AD5259 Digital Potentiometers.  These parts are
very similar to the AD5246 that I already had but they are in slightly
bigger packages and have I2C address pins so I can get more than 1 on
the same I2C bus without a MUX.  Also added some current sensing
resistors that are rated for 1A at .1ohms and 1% tolerance.  These will
possibly go with the INA219 assuming I can get 5 of these parts onto the
I2C bus.  Otherwise I need to either cut them out of the design or go
back to the I2C MUX idea.
Parts:
- added JP18: (no value), SparkFun-Connectors:1X05
- added R10, R6, R7, R8, R9: (no value), SparkFun-Resistors:R2010
- added U$2: AD5245SOT23-8, Mikes-Stuff:SOT23-8
- added U$3: AD5259MSOP-10, Mikes-Stuff:MSOP-10
- moved U13 187.1 mm to (95.2, 26.7)
Connections:
- new net N$1: U$2.8
- new net N$10: U$2.1
- new net N$14: U$2.2
- new net N$15: U$2.3
- new net N$16: U$2.4
- new net N$17: U$3.1
- new net N$18: U$3.2
- new net N$19: U$3.3
- new net N$20: U$3.4
- new net N$21: U$3.5
- new net N$22: U$3.6
- new net N$23: U$3.7
- new net N$26: U$3.8
- new net N$27: U$3.9
- new net N$29: U$3.10
- new net N$4: U$2.7
- new net N$5: U$2.6
- new net N$8: U$2.5
- net 5V: now also JP18.4
- net GND: now also JP18.3
- net RES: now also JP18.5
- net SCL: now also JP18.1
- net SDA: now also JP18.2

Commit message: FishLight_PCB: Added the AD5248 digital pot symbol
Added the AD5248 digital potentiometer.  This pot has 2 circuits and 2
address pins.  By getting 3 of these parts, I will be able to
individually select each LED channels current limit with 1 extra
potentiometer without having to use a MUX.  This saves space, potential
noise issues, and some cost.  I have not yet added this pot to the
schematic, only to the library.
Parts:
- removed U$2: AD5245SOT23-8, Mikes-Stuff:SOT23-8
- removed U$3: AD5259MSOP-10, Mikes-Stuff:MSOP-10
Connections:
- removed net N$1: U$2.8
- removed net N$10: U$2.1
- removed net N$14: U$2.2
- removed net N$15: U$2.3
- removed net N$16: U$2.4
- removed net N$17: U$3.1
- removed net N$18: U$3.2
- removed net N$19: U$3.3
- removed net N$20: U$3.4
- removed net N$21: U$3.5
- removed net N$22: U$3.6
- removed net N$23: U$3.7
- removed net N$26: U$3.8
- removed net N$27: U$3.9
- removed net N$29: U$3.10
- removed net N$4: U$2.7
- removed net N$5: U$2.6
- removed net N$8: U$2.5
Changed lines of the file:
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@@
 <element name="R5" library="SparkFun-Resistors" package="0603-RES" value="4.7K" x="-90.17" y="-274.32"/>
 <element name="JP18" library="SparkFun-Connectors" package="1X05" value="" x="-88.9" y="-280.67"/>
-<element name="U$2" library="Mikes-Stuff" package="SOT23-8" value="AD5245SOT23-8" x="97.79" y="12.7"/>
-<element name="U$3" library="Mikes-Stuff" package="MSOP-10" value="AD5259MSOP-10" x="91.44" y="13.97"/>
 <element name="R6" library="SparkFun-Resistors" package="R2010" value="" x="-87.63" y="-284.48"/>
 <element name="R7" library="SparkFun-Resistors" package="R2010" value="" x="-87.63" y="-288.29"/>
@@
 <contactref element="U$1" pad="13"/>
 </signal>
-<signal name="N$1">
-<contactref element="U$2" pad="8"/>
-</signal>
-<signal name="N$4">
-<contactref element="U$2" pad="7"/>
-</signal>
-<signal name="N$5">
-<contactref element="U$2" pad="6"/>
-</signal>
-<signal name="N$8">
-<contactref element="U$2" pad="5"/>
-</signal>
-<signal name="N$10">
-<contactref element="U$2" pad="1"/>
-</signal>
-<signal name="N$14">
-<contactref element="U$2" pad="2"/>
-</signal>
-<signal name="N$15">
-<contactref element="U$2" pad="3"/>
-</signal>
-<signal name="N$16">
-<contactref element="U$2" pad="4"/>
-</signal>
-<signal name="N$17">
-<contactref element="U$3" pad="1"/>
-</signal>
-<signal name="N$18">
-<contactref element="U$3" pad="2"/>
-</signal>
-<signal name="N$19">
-<contactref element="U$3" pad="3"/>
-</signal>
-<signal name="N$20">
-<contactref element="U$3" pad="4"/>
-</signal>
-<signal name="N$21">
-<contactref element="U$3" pad="5"/>
-</signal>
-<signal name="N$22">
-<contactref element="U$3" pad="6"/>
-</signal>
-<signal name="N$23">
-<contactref element="U$3" pad="7"/>
-</signal>
-<signal name="N$26">
-<contactref element="U$3" pad="8"/>
-</signal>
-<signal name="N$27">
-<contactref element="U$3" pad="9"/>
-</signal>
-<signal name="N$29">
-<contactref element="U$3" pad="10"/>
-</signal>
 </signals>

Commit message: FishLight_PCB: Connected the AD5248
Replaced the existing potentiometers with the AD5248.  Set addresses 00,
01, and 10.
Parts:
- removed C10, C11, C13: 0.1uF, SparkFun-Capacitors:0603-CAP
- removed U10, U11, U12, U13, U9: AD5246TSSOT6, Mikes-Stuff:TSSOT6
- removed U8: CD74HC4067SSOP24, Mikes-Stuff:SSOP24
- added U$2, U$3, U$4: AD5248MSOP-10, Mikes-Stuff:MSOP-10
Connections:
- removed net N$11: U8.10
- removed net N$12: U8.11
- removed net N$24: U8.13
- removed net N$25: U8.14
- removed net N$28: U8.15
- removed net N$9: U8.4
- removed net SDA1: U8.9, U9.4
- removed net SDA2: U10.4, U8.8
- removed net SDA3: U11.4, U8.7
- removed net SDA4: U12.4, U8.6
- removed net SDA5: U13.4, U8.5
- net 5V: now also C7.2, C8.2, C9.2, U$2.5, U$3.5, U$3.8, U$4.2, U$4.5; no longer C10.1, C11.1, C13.2, C7.1, C8.1, C9.1, U10.1, U11.1, U12.1, U13.1, U8.24, U9.1
- net GND: now also C7.1, C8.1, C9.1, U$2.1, U$2.2, U$2.4, U$2.8, U$2.9, U$3.1, U$3.2, U$3.4, U$3.9, U$4.1, U$4.4, U$4.8, U$4.9; no longer C10.2, C11.2, C13.1, C7.2, C8.2, C9.2, U10.2, U10.6, U11.2, U11.6, U12.2, U12.6, U13.2, U13.6, U8.12, U9.2, U9.6
- net LR1: now also U$2.3; no longer U9.5
- net LR2: now also U$2.10; no longer U10.5
- net LR3: now also U$3.3; no longer U11.5
- net LR4: now also U$3.10; no longer U12.5
- net LR5: now also U$4.3; no longer U13.5
- net SCL: now also U$2.6, U$3.6, U$4.6; no longer U10.3, U11.3, U12.3, U13.3, U9.3
- net SDA: now also U$2.7, U$3.7, U$4.7; no longer U8.1

Commit message: FishLight_PCB: Initial part placement
Did an initial placement of the main components (LED drivers,
potentiometers, LED screw terminals, voltage regulators) to get an idea
of how they may fit together.  Also removed the extra screw terminals.
Although I like this idea as a developer, I think there just isn't
enough space or need for them in this project.
Parts:
- removed JP13, JP14, JP15, JP16, JP17, JP4, JP5, JP6, JP7, JP8: (no value), Mikes-Stuff:SCREWTERMINAL-3.5MM-3
- moved U$2 355.9 mm to (35.6, 34.3), turned to 270 degrees
- moved U$3 347.7 mm to (35.6, 22.9), turned to 90 degrees
- moved U$4 337.5 mm to (35.6, 8.89), turned to 270 degrees
- moved U15 335.9 mm to (74.9, 49.5), turned to 180 degrees
- moved JP9 270.3 mm to (80.0, 24.1), turned to 90 degrees
- moved JP10 267.0 mm to (80.0, 12.4), turned to 90 degrees
- moved JP12 262.3 mm to (5.08, 30.5), turned to 270 degrees
- moved JP11 244.0 mm to (5.08, 18.8), turned to 270 degrees
- moved U14 240.4 mm to (74.9, 74.9)
- moved U5 83.6 mm to (50.8, 24.1), turned to 270 degrees
- moved U4 77.8 mm to (50.8, 36.8), turned to 270 degrees
- moved U7 72.8 mm to (20.3, 7.62), turned to 90 degrees
- moved U6 64.3 mm to (20.3, 20.3), turned to 90 degrees
- moved U3 42.4 mm to (20.3, 33.0), turned to 90 degrees
- moved U2 19.2 mm to (26.7, 66.0)
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Connections:
- removed net 3.3V: JP13.1, JP14.1
- removed net AREF: JP15.3
- removed net D12: JP8.3
- removed net D13: JP8.2
- removed net D8: JP6.1
- new net N$14: U$4.1
- new net N$17: U$4.9
- net 12V: no longer JP15.1
- net 5V: no longer JP13.3, JP14.3
- net A0: no longer JP17.3
- net A1: no longer JP17.2
- net A2: no longer JP17.1
- net A3: no longer JP16.3
- net D10: no longer JP7.2
- net D11: no longer JP7.1
- net D2: no longer JP4.1
- net D3: no longer JP5.3
- net D4: no longer JP5.2
- net D5: no longer JP5.1
- net D6: no longer JP6.3
- net D7: no longer JP6.2
- net D9: no longer JP7.3
- net GND: no longer JP13.2, JP14.2, JP8.1, U$4.1, U$4.9
- net RES: no longer JP15.2
- net RX: no longer JP4.2
- net SCL: no longer JP16.1
- net SDA: no longer JP16.2
- net TX: no longer JP4.3
Other:
- board text added: "Vias to gnd"
- board text removed: "3.3V"
- board text removed: "5V"
- board text removed: "A0"
- board text removed: "A1"
- board text removed: "A2"
- board text removed: "A3"
- board text removed: "A4"
- board text removed: "A5"
- board text removed: "Aref"
- board text removed: "BL"
- board text removed: "CW"
- board text removed: "D0"
- board text removed: "D1"
- board text removed: "D10*"
- board text removed: "D11*"
- board text removed: "D12"
- board text removed: "D13"
- board text removed: "D2"
- board text removed: "D3*"
- board text removed: "D4"
- board text removed: "D5*"
- board text removed: "D6*"
- board text removed: "D7"
- board text removed: "D8"
- board text removed: "D9*"
- board text removed: "GND"
- board text removed: "LED GND"
- board text removed: "Rst"
- board text removed: "Vin"
- board text removed: "WW"

Commit message: FishLight_PCB: Added INA219 current sensor
Added the INA219 current sensor.  This will make sure that I am driving
the LEDs with the amount of current I am expecting.  I can also use this
to hone in on my potentiometer settings.  These are removable if the
board gets too crowded.
Parts:
- added C10, C11, C13, C16, C17: 0.1uF, SparkFun-Capacitors:0603-CAP
- added U$5, U$6, U$7, U$8, U$9: INA219SOT23-8, Mikes-Stuff:SOT23-8
- moved JP18 354.2 mm to (39.4, 49.5), turned to 180 degrees
- moved R5 339.8 mm to (69.8, 25.4)
- moved R4 335.3 mm to (69.8, 22.9)
- moved R3 334.2 mm to (69.8, 24.1)
- moved R10 330.2 mm to (11.4, 15.2)
- moved R6 330.2 mm to (11.4, 30.5)
- moved R7 330.2 mm to (11.4, 26.7)
- moved R8 330.2 mm to (11.4, 22.9)
- moved R9 330.2 mm to (11.4, 19.1)
- moved C15 330.1 mm to (66.0, 25.4)
- moved C14 327.9 mm to (66.0, 26.7)
- moved JP1 230.2 mm to (7.62, 74.9)
- moved JP2 230.2 mm to (7.62, 68.6)
- moved JP3 230.2 mm to (7.62, 62.2)
- moved C12 211.1 mm to (66.0, 20.3)
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Connections:
- net 24V: now also R10.2, R6.2, R7.2, R8.2, R9.2, U$5.1, U$6.1, U$7.1, U$8.1, U$9.1
- net 5V: now also C10.2, C11.2, C13.2, C16.2, C17.2, U$5.4, U$6.4, U$7.4, U$8.4, U$9.4, U$9.8
- net GND: now also C10.1, C11.1, C13.1, C16.1, C17.1, U$5.3, U$6.3, U$7.3, U$8.3, U$8.8, U$9.3, U$9.7
- net LED1: now also R6.1, U$5.2
- net LED2: now also R7.1, U$6.2
- net LED3: now also R8.1, U$7.2
- net LED4: now also R9.1, U$8.2
- net LED5: now also R10.1, U$9.2
- net SCL: now also U$8.5, U$8.7, U$9.5
- net SDA: now also U$8.6, U$9.6

Commit message: FishLight_PCB: Added fans and moved parts around
Moved parts around on the board to be a bit more friendly to the 24V
rail.  Also changed the color of the top silk screen layer but I doubt
that will stick.  Added some fan connectors in the hopes that I can add
a 3 pin fan in the future.  Need to come up with a good control circuit
for that tho.  I would like to have speed control not just on and off.
Parts:
- removed U$1: SPARK_CORECORE, Spark:SPARK_CORE
- removed U$2, U$3, U$4: AD5248MSOP-10, Mikes-Stuff:MSOP-10
- removed U$5, U$6, U$7, U$8, U$9: INA219SOT23-8, Mikes-Stuff:SOT23-8
- added JP4, JP5: (no value), SparkFun-Connectors:MOLEX-1X3
- added JP6, JP7: M023.5MM, SparkFun-Connectors:SCREWTERMINAL-3.5MM-2
- added U1: SPARK_CORECORE, Spark:SPARK_CORE
- added U10, U8, U9: AD5248MSOP-10, Mikes-Stuff:MSOP-10
- added U11, U12, U13: INA219SOT23-8, Mikes-Stuff:SOT23-8
- added U16: UA7812D2PAK-3, Mikes-Stuff:D2PAK-3
- added U17: L7805D2PAK-2, Mikes-Stuff:D2PAK-2
- U14: value UA7812D2PAK-3 -> INA219SOT23-8; device Mikes-Stuff:D2PAK-3 -> Mikes-Stuff:SOT23-8
- U15: value L7805D2PAK-2 -> INA219SOT23-8; device Mikes-Stuff:D2PAK-2 -> Mikes-Stuff:SOT23-8
- moved U14 84.5 mm to (12.7, 17.8)
- moved U15 73.6 mm to (12.7, 10.2), turned to 0 degrees
- moved R1 44.0 mm to (94.0, 58.4)
- moved R2 44.0 mm to (94.0, 57.1)
- moved R3 44.0 mm to (94.0, 61.0)
- moved R4 44.0 mm to (94.0, 59.7)
- moved R5 44.0 mm to (94.0, 62.2)
- moved C1 44.0 mm to (90.2, 58.4)
- moved C11 44.0 mm to (90.2, 68.6)
- moved C12 44.0 mm to (90.2, 57.1)
- moved C13 44.0 mm to (90.2, 67.3)
- moved C14 44.0 mm to (90.2, 63.5)
- moved C15 44.0 mm to (90.2, 62.2)
- moved C16 44.0 mm to (90.2, 66.0)
- moved C17 44.0 mm to (90.2, 64.8)
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Connections:
- removed net D10: U4.1
- removed net D11: U5.1
- removed net D9: U3.1
- removed net N$13: JP1.2, R5.1
- removed net N$2: JP3.2, R3.1
- removed net N$7: JP2.2, R4.1
- net 12V: now also JP4.2, JP5.2, U16.3; no longer U14.3
- net 24V: now also JP6.1, JP6.2, U11.1, U12.1, U13.1, U16.1, U17.1; no longer U$5.1, U$6.1, U$7.1, U$8.1, U$9.1
- net 5V: now also U1.24, U10.2, U10.5, U11.4, U12.4, U13.4, U14.4, U15.4, U15.8, U17.3, U8.5, U9.5, U9.8; no longer U$1.24, U$2.5, U$3.5, U$3.8, U$4.2, U$4.5, U$5.4, U$6.4, U$7.4, U$8.4, U$9.4, U$9.8, U15.3
- net A0: now also U1.12; no longer U$1.12
- net A1: now also U1.11; no longer U$1.11
- net A2: now also U1.10; no longer U$1.10
- net A3: now also U1.9; no longer U$1.9
- net A6: now also U1.6; no longer U$1.6
- net A7: now also U1.5; no longer U$1.5
- net D0: now also U1.13, U3.1; no longer U$1.13
- net D1: now also U1.14, U4.1; no longer U$1.14
- net D2: now also U1.15, U5.1; no longer U$1.15
- net D3: now also U1.16; no longer U$1.16
- net D4: now also U1.17, U7.1; no longer U$1.17
- net D5: now also JP1.2, JP2.2, JP3.2, R3.1, R4.1, R5.1, U1.18; no longer U$1.18, U7.1
- net D6: now also U1.19; no longer U$1.19
- net D7: now also U1.20; no longer U$1.20
- net GND: now also JP4.1, JP5.1, JP7.1, JP7.2, U1.2, U1.21, U10.4, U10.8, U11.3, U12.3, U13.3, U14.3, U14.8, U15.3, U15.7, U16.2, U17.2, U8.1, U8.2, U8.4, U8.8, U8.9, U9.1, U9.2, U9.4, U9.9; no longer U$1.2, U$1.21, U$2.1, U$2.2, U$2.4, U$2.8, U$2.9, U$3.1, U$3.2, U$3.4, U$3.9, U$4.4, U$4.8, U$5.3, U$6.3, U$7.3, U$8.3, U$8.8, U$9.3, U$9.7, U14.2, U15.2
- net LED1: now also U11.2; no longer U$5.2
- net LED2: now also U12.2; no longer U$6.2
- net LED3: now also U13.2; no longer U$7.2
- net LED4: now also U14.2; no longer U$8.2
- net LED5: now also U15.2; no longer U$9.2
- net LR1: now also U8.3; no longer U$2.3
- net LR2: now also U8.10; no longer U$2.10
- net LR3: now also U9.3; no longer U$3.3
- net LR4: now also U9.10; no longer U$3.10
- net LR5: now also U10.3; no longer U$4.3
- net N$14: now also U10.1; no longer U$4.1
- net N$17: now also U10.9; no longer U$4.9
- net RAW: now also U1.1; no longer U$1.1
- net RES: now also U1.23; no longer U$1.23
- net RX: now also U1.4; no longer U$1.4
- net SCL: now also U1.8, U10.6, U14.5, U14.7, U15.5, U8.6, U9.6; no longer U$1.8, U$2.6, U$3.6, U$4.6, U$8.5, U$8.7, U$9.5
- net SDA: now also U1.7, U10.7, U14.6, U15.6, U8.7, U9.7; no longer U$1.7, U$2.7, U$3.7, U$4.7, U$8.6, U$9.6
- net TX: now also U1.3; no longer U$1.3
- net VDDA: now also U1.22; no longer U$1.22
Other:
- board text added: "12V"
- board text added: "Fans"
- board text added: "GND"
- board text added: "Temp Sensors"
