File: FishLight-v01.brd (EAGLE design)
At the start: 85.1 x 85.1 mm, 61 parts, among them U1 SPARK_CORECORE, U10 AD5248MSOP-10, U11 INA219SOT23-8, U12 INA219SOT23-8, U13 INA219SOT23-8, U14 INA219SOT23-8, U15 INA219SOT23-8, U16 UA7812D2PAK-3, U17 L7805D2PAK-2, U2 RTCBREAKOUT, U3 CAT4101TO-263, U4 CAT4101TO-263, U5 CAT4101TO-263, U6 CAT4101TO-263, U7 CAT4101TO-263, U8 AD5248MSOP-10, U9 AD5248MSOP-10

Commit message: FishLight_PCB: Added power headers
Added some single pin headers for the power rails.  Also moved
the current sensing resistors to the back of the board.
Hopefully this will help me route the control signals a little
easier.
Parts:
- removed R3, R5: 4.7K, SparkFun-Resistors:0603-RES
- added JP13, JP14, JP15, JP8: M01PTH, SparkFun-Connectors:1X01
- moved R10 9.00 mm to (12.7, 15.3), flipped to the bottom, turned to 180 degrees
- moved U11 7.00 mm to (12.7, 33.6)
- moved R6 6.00 mm to (12.7, 30.8), flipped to the bottom, turned to 180 degrees
- moved U15 5.00 mm to (12.7, 15.2)
- moved R9 4.90 mm to (12.7, 18.9), flipped to the bottom, turned to 180 degrees
- moved U12 4.00 mm to (12.7, 29.0)
- moved R7 2.00 mm to (12.7, 27.2), flipped to the bottom, turned to 180 degrees
- moved R8 2.00 mm to (12.7, 23.6), flipped to the bottom, turned to 180 degrees
- moved U14 2.00 mm to (12.7, 19.8)
- moved U13 1.00 mm to (12.7, 24.4)
Connections:
- net 12V: now also JP15.1
- net 24V: now also JP13.1
- net 5V: now also JP8.1; no longer R3.2, R5.2
- net D5: no longer R3.1, R5.1
- net GND: now also JP14.1

Commit message: FishLight_PCB: Start wires for current sensor
Started routing some wires for the 24V rail and the current sense
components.  There is a very large 24V trace and some vias connecting
the resistors on the bottom to the sensor on the top.
Parts:
- moved JP13 13.6 mm to (16.0, 37.0)
- moved U11 2.31 mm to (12.3, 31.4), turned to 180 degrees
- moved U12 2.08 mm to (12.3, 27.0), turned to 180 degrees
- moved U13 1.84 mm to (12.3, 22.6), turned to 180 degrees
- moved U14 1.61 mm to (12.3, 18.2), turned to 180 degrees
- moved U15 1.38 mm to (12.3, 13.8), turned to 180 degrees
- moved JP8 1.00 mm to (8.00, 50.0)
Routing:
- net 24V: track 0.00 -> 47.8 mm

Commit message: FishLight_PCB: Added the RK7002B N-MOSFET
Added the RK7002B N-Channel MOSFET.  This will allow me to turn on and
off the 2 fans that I have connectors for.
Parts:
- added R3, R5: 10K, SparkFun-Resistors:0603-RES
- added U18, U19: RK7002BSOT23-3, Mikes-Stuff:SOT-23-3
- moved R4 92.0 mm to (2.31, 68.0), turned to 90 degrees
- moved R2 49.0 mm to (46.0, 67.2)
- moved R1 48.4 mm to (46.0, 64.4)
- moved U10 18.3 mm to (52.9, 6.38), turned to 90 degrees
- moved U7 12.3 mm to (68.1, 7.65), turned to 270 degrees
- moved U3 4.00 mm to (38.1, 37.0)
- moved U4 4.00 mm to (68.6, 38.3)
- moved U8 4.00 mm to (53.3, 35.8)
- moved JP3 2.00 mm to (7.62, 60.2)
- moved JP2 1.00 mm to (7.62, 67.6)
- moved JP4 1.00 mm to (20.3, 69.6)
Connections:
- new net FAN1: U18.2
- new net FAN2: U19.2
- new net N$1: JP5.1, R5.2, U19.3
- new net N$15: JP4.1, R3.2, U18.3
- net GND: now also R3.1, R5.1, U18.1, U19.1; no longer JP4.1, JP5.1
Routing:
- net 24V: track 47.8 -> 51.4 mm
Other:
- board text added: "24V"
- board text removed: "12V"

Commit message: FishLight_PCB: Fixed fan transistors
Fixed the fan connector transistor pull down resistors.  These were
connected to drain but they need to be connected to gate so that the
transistor shuts off correctly.  Also added some Solid State Relays to
possibly turn on and off some AC loads (such as a pump or the heater)
for emergency situations.  These will probably go away though.  Kind of
an interesting idea is all.
Parts:
- added R11, R12: 10K, SparkFun-Resistors:0603-RES
- added U20, U21: RELAY-SOLIDSTATEPTH, SparkFun-Electromechanical:RELAY-S108T02
- R1, R2: value 10K -> 4.7K
- moved R3 2.00 mm to (26.0, 75.0), turned to 180 degrees
- moved R5 1.00 mm to (26.0, 57.0), turned to 180 degrees
Connections:
- new net N$16: R11.1, U19.3
- new net N$18: JP5.1, R11.2
- net FAN1: now also R3.2
- net FAN2: now also R5.2
- net N$1: now also JP4.1, R12.2; no longer JP5.1, R5.2, U19.3
- net N$15: now also R12.1; no longer JP4.1, R3.2
Changed lines of the file:
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@@
 <attribute name="VALUE" x="89.154" y="48.387" size="0.4064" layer="27" font="vector"/>
 </element>
-<element name="R1" library="SparkFun-Resistors" package="0603-RES" value="10K" x="45.98" y="64.42" smashed="yes">
+<element name="R1" library="SparkFun-Resistors" package="0603-RES" value="4.7K" x="45.98" y="64.42" smashed="yes">
 <attribute name="NAME" x="45.091" y="65.182" size="0.4064" layer="25" font="vector"/>
 <attribute name="VALUE" x="44.964" y="63.277" size="0.4064" layer="27" font="vector"/>
 </element>
-<element name="R2" library="SparkFun-Resistors" package="0603-RES" value="10K" x="45.98" y="67.15" smashed="yes">
+<element name="R2" library="SparkFun-Resistors" package="0603-RES" value="4.7K" x="45.98" y="67.15" smashed="yes">
 <attribute name="NAME" x="45.091" y="67.912" size="0.4064" layer="25" font="vector"/>
 <attribute name="VALUE" x="44.964" y="66.007" size="0.4064" layer="27" font="vector"/>
@@
 <element name="U18" library="Mikes-Stuff" package="SOT-23-3" value="RK7002BSOT23-3" x="22" y="75"/>
 <element name="U19" library="Mikes-Stuff" package="SOT-23-3" value="RK7002BSOT23-3" x="22" y="57"/>
-<element name="R3" library="SparkFun-Resistors" package="0603-RES" value="10K" x="26" y="77"/>
-<element name="R5" library="SparkFun-Resistors" package="0603-RES" value="10K" x="26" y="58"/>
+<element name="R3" library="SparkFun-Resistors" package="0603-RES" value="10K" x="26" y="75" rot="R180"/>
+<element name="R5" library="SparkFun-Resistors" package="0603-RES" value="10K" x="26" y="57" rot="R180"/>
+<element name="U20" library="SparkFun-Electromechanical" package="RELAY-S108T02" value="RELAY-SOLIDSTATEPTH" x="94" y="13" rot="R90"/>
+<element name="U21" library="SparkFun-Electromechanical" package="RELAY-S108T02" value="RELAY-SOLIDSTATEPTH" x="89" y="13" rot="R90"/>
+<element name="R11" library="SparkFun-Resistors" package="0603-RES" value="10K" x="18" y="59" rot="R90"/>
+<element name="R12" library="SparkFun-Resistors" package="0603-RES" value="10K" x="19" y="75" rot="R90"/>
 </elements>
 <signals>
@@
 <wire x1="17" y1="50" x2="12" y2="32.56" width="0" layer="19" extent="1-1"/>
 <wire x1="22.95" y1="55.95" x2="17" y2="50" width="0" layer="19" extent="1-1"/>
-<wire x1="25.15" y1="58" x2="22.95" y2="55.95" width="0" layer="19" extent="1-1"/>
+<wire x1="26.85" y1="57" x2="22.95" y2="55.95" width="0" layer="19" extent="1-1"/>
 <wire x1="7.62" y1="60.23" x2="17" y2="50" width="0" layer="19" extent="1-1"/>
 <wire x1="7.62" y1="67.58" x2="7.62" y2="60.23" width="0" layer="19" extent="1-1"/>
 <wire x1="7.62" y1="74.93" x2="7.62" y2="67.58" width="0" layer="19" extent="1-1"/>
 <wire x1="22.95" y1="73.95" x2="7.62" y2="74.93" width="0" layer="19" extent="1-1"/>
-<wire x1="25.15" y1="77" x2="22.95" y2="73.95" width="0" layer="19" extent="1-1"/>
+<wire x1="26.85" y1="75" x2="22.95" y2="73.95" width="0" layer="19" extent="1-1"/>
 </signal>
 <signal name="5V" airwireshidden="yes">
@@
 <via x="10.3" y="15.4" extent="1-16" drill="0.508" shape="square"/>
 </signal>
-<signal name="N$1">
-<contactref element="JP5" pad="1"/>
-<contactref element="U19" pad="3"/>
-<contactref element="R5" pad="2"/>
-<wire x1="22" y1="58.05" x2="20.32" y2="62.23" width="0" layer="19" extent="1-1"/>
-<wire x1="26.85" y1="58" x2="22" y2="58.05" width="0" layer="19" extent="1-1"/>
-</signal>
-<signal name="N$15">
-<contactref element="JP4" pad="1"/>
-<contactref element="U18" pad="3"/>
-<contactref element="R3" pad="2"/>
-<wire x1="22" y1="76.05" x2="26.85" y2="77" width="0" layer="19" extent="1-1"/>
-<wire x1="20.32" y1="69.58" x2="22" y2="76.05" width="0" layer="19" extent="1-1"/>
-</signal>
 <signal name="FAN2">
 <contactref element="U19" pad="2"/>
+<contactref element="R5" pad="2"/>
+<wire x1="21.05" y1="55.95" x2="25.15" y2="57" width="0" layer="19" extent="1-1"/>
 </signal>
 <signal name="FAN1">
 <contactref element="U18" pad="2"/>
+<contactref element="R3" pad="2"/>
+<wire x1="21.05" y1="73.95" x2="25.15" y2="75" width="0" layer="19" extent="1-1"/>
+</signal>
+<signal name="N$1">
+<contactref element="JP4" pad="1"/>
+<contactref element="R12" pad="2"/>
+<wire x1="19" y1="75.85" x2="20.32" y2="69.58" width="0" layer="19" extent="1-1"/>
+</signal>
+<signal name="N$15">
+<contactref element="R12" pad="1"/>
+<contactref element="U18" pad="3"/>
+<wire x1="19" y1="74.15" x2="22" y2="76.05" width="0" layer="19" extent="1-1"/>
+</signal>
+<signal name="N$16">
+<contactref element="U19" pad="3"/>
+<contactref element="R11" pad="1"/>
+<wire x1="18" y1="58.15" x2="22" y2="58.05" width="0" layer="19" extent="1-1"/>
+</signal>
+<signal name="N$18">
+<contactref element="R11" pad="2"/>
+<contactref element="JP5" pad="1"/>
+<wire x1="18" y1="59.85" x2="20.32" y2="62.23" width="0" layer="19" extent="1-1"/>
 </signal>
 </signals>

Commit message: FishLight_PCB: Moved Current Sensor resistor vias
The Vias that connect the current sensor resistors to the top layer were
not centered very well on their pads.  This should help to distribute
the current a bit better.
Parts:
- moved JP13 0.77 mm to (15.2, 36.9)
Routing:
- net 24V: track 51.4 -> 18.6 mm
- net N$19: track 0.00 -> 32.8 mm

Commit message: FishLight_PCB: Added LED strings 4 - 8
Added LED strings 4 - 8 and removed the 'green' string.  This will allow
me to control 2 tanks or one really big tank in the future.  Added all
of the accompanying parts and moved a lot of stuff around to make it all
fit on the schematic.  Still need to lay them out on the board tho.
Parts:
- added C18, C19, C20, C21, C22, C23, C24: 0.1uF, SparkFun-Capacitors:0603-CAP
- added JP16, JP20: (no value), Mikes-Stuff:SCREWTERMINAL-3.5MM-3
- added R13, R14, R15: (no value), SparkFun-Resistors:R2010
- added U22: AD5248MSOP-10, Mikes-Stuff:MSOP-10
- added U23, U24, U25: CAT4101TO-263, Mikes-Stuff:TO-263
- added U26, U27, U28: INA219SOT23-8, Mikes-Stuff:SOT23-8
Connections:
- removed net N$14: U10.1
- removed net N$17: U10.9
- removed net N$3: JP11.3
- removed net N$6: JP10.1
- new net LED6: JP11.3, R13.1, U26.2
- new net LED7: JP20.1, R14.1, U27.2
- new net LED8: JP20.2, R15.1, U28.2
- new net LG6: JP10.1, U23.5
- new net LG7: JP16.3, U25.5
- new net LG8: JP16.2, U24.5
- new net LR6: U10.10, U23.4
- new net LR7: U22.3, U25.4
- new net LR8: U22.10, U24.4
- new net N$22: JP20.3
- new net N$27: JP16.1
- net 24V: now also R13.2, R14.2, R15.2, U26.1, U27.1, U28.1
- net 5V: now also C18.2, C19.1, C20.1, C21.1, C22.2, C23.2, C24.2, U12.7, U22.2, U22.5, U22.8, U23.2, U24.2, U25.2, U26.4, U26.7, U26.8, U27.4, U27.8, U28.4, U28.8
- net D0: now also U7.1
- net D1: now also U23.1
- net D2: now also U25.1
- net D3: now also U24.1
- net D4: no longer U7.1
- net GND: now also C18.1, C19.2, C20.2, C21.2, C22.1, C23.1, C24.1, U10.1, U10.9, U11.7, U11.8, U12.8, U13.8, U22.1, U22.4, U22.9, U23.3, U23.6, U24.3, U24.6, U25.3, U25.6, U26.3, U27.3, U28.3
- net SCL: now also U11.5, U12.5, U13.5, U22.6, U26.5, U27.5, U28.5, U28.7
- net SDA: now also U11.6, U12.6, U13.6, U13.7, U22.7, U26.6, U27.6, U27.7, U28.6
Other:
- board text added: "MAKE THIS BIGGER"

Commit message: FishLight_PCB: Replaced the RTC and added VIAs
Replaced the giant RTC breakout board with the new DS3231M RTC.  This
can fit right under the Spark Core so it takes up very little space.
The battery is still kinda big but its not a big deal.  Also added VIAs
to the CAT4101s that are on the top side and to the I-Sense resistors
that are new.
Parts:
- removed U2: RTCBREAKOUT, Mikes-Stuff:RTCBREAKOUT
- added BAT1: (no value), SparkFun-Electromechanical:BATTCON_12MM_PTH
- added C25: 0.1uF, SparkFun-Capacitors:0603-CAP
- added U29: DS3231MSOIC-8, Mikes-Stuff:SOIC-8
- moved C22 227.8 mm to (90.0, 71.0)
- moved C23 226.8 mm to (90.0, 72.0)
- moved C24 225.8 mm to (90.0, 73.0)
- moved C21 191.1 mm to (90.0, 45.0), flipped to the bottom
- moved R14 167.6 mm to (12.6, 39.0), flipped to the bottom, turned to 180 degrees
- moved R15 162.2 mm to (12.6, 34.7), flipped to the bottom, turned to 180 degrees
- moved U28 159.6 mm to (12.3, 35.9), turned to 180 degrees
- moved U27 158.4 mm to (12.3, 40.6), turned to 180 degrees
- moved U25 154.8 mm to (69.0, 34.0), flipped to the bottom, turned to 90 degrees
- moved C19 147.3 mm to (90.0, 47.0), flipped to the bottom
- moved C20 144.0 mm to (90.0, 46.0), flipped to the bottom
- moved R13 134.9 mm to (12.7, 11.8), flipped to the bottom, turned to 180 degrees
- moved U26 128.6 mm to (12.3, 9.19), turned to 180 degrees
- moved C18 123.9 mm to (90.0, 48.0), flipped to the bottom, turned to 180 degrees
- moved U24 120.8 mm to (38.2, 34.4), flipped to the bottom, turned to 270 degrees
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Connections:
- removed net N$22: JP20.3
- removed net N$27: JP16.1
- new net N$3: BAT1.VCC@1, U29.6
- net 5V: now also C25.1, U29.2; no longer U2.5
- net GND: now also BAT1.GND, C25.2, U29.5; no longer U2.4
- net LED7: now also JP20.2; no longer JP20.1
- net LED8: now also JP20.3; no longer JP20.2
- net LG7: now also JP16.2; no longer JP16.3
- net LG8: now also JP16.1; no longer JP16.2
- net SCL: now also U29.8; no longer U2.2
- net SDA: now also U29.7; no longer U2.1
- net SQW: now also U29.3; no longer U2.3
Routing:
- net N$19: track 32.8 -> 41.8 mm

Commit message: FishLight_PCB: Swapped out the LCD connector
The LCD connector was just a 5pin header.  Now it is a polarized header
so that it cannot be plugged in backwards on accident.  Also moved some
things around to get straighter lines on the I2C bus.
Parts:
- JP18: device SparkFun-Connectors:1X05 -> Mikes-Stuff:MOLEX-1X5
- moved R1 10.0 mm to (54.0, 58.4)
- moved R2 9.44 mm to (49.6, 58.4), turned to 180 degrees
- moved C25 3.16 mm to (50.0, 52.0)
- moved U29 3.16 mm to (54.0, 52.0)
- moved JP10 2.00 mm to (80.0, 10.4)
- moved JP16 2.00 mm to (80.0, 33.7)
- moved JP9 2.00 mm to (80.0, 22.1)
- moved JP18 1.00 mm to (50.2, 66.8)
