File: FishLight-v01.sch (EAGLE design)
At the start: 63 parts, among them U1 SPARK_CORECORE, U10 AD5248MSOP-10, U11 INA219SOT23-8, U12 INA219SOT23-8, U13 INA219SOT23-8, U14 INA219SOT23-8, U15 INA219SOT23-8, U16 UA7812D2PAK-3, U17 L7805D2PAK-2, U2 RTCBREAKOUT, U3 CAT4101TO-263, U4 CAT4101TO-263, U5 CAT4101TO-263, U6 CAT4101TO-263, U7 CAT4101TO-263, U8 AD5248MSOP-10, U9 AD5248MSOP-10

Commit message: FishLight_PCB: Added the RK7002B N-MOSFET
Added the RK7002B N-Channel MOSFET.  This will allow me to turn on and
off the 2 fans that I have connectors for.
Parts:
- added R3, R5: 10K, SparkFun-Resistors:RESISTOR0603-RES
- added U18, U19: RK7002BSOT23-3, Mikes-Stuff:RK7002BSOT23-3
Connections:
- new net FAN1: U18.G
- new net FAN2: U19.G
- new net N$1: JP5.1, R5.2, U19.D
- new net N$15: JP4.1, R3.2, U18.D
- net GND: now also R3.1, R5.1, U18.S, U19.S; no longer JP4.1, JP5.1
Other:
- note added: "Screws"
- moved on the sheet: JP4
Changed lines of the file:
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@@
 <part name="JP14" library="SparkFun-Connectors" deviceset="M01" device="PTH"/>
 <part name="JP15" library="SparkFun-Connectors" deviceset="M01" device="PTH"/>
+<part name="U18" library="Mikes-Stuff" deviceset="RK7002B" device="SOT23-3"/>
+<part name="U19" library="Mikes-Stuff" deviceset="RK7002B" device="SOT23-3"/>
+<part name="R3" library="SparkFun-Resistors" deviceset="RESISTOR" device="0603-RES" value="10K"/>
+<part name="R5" library="SparkFun-Resistors" deviceset="RESISTOR" device="0603-RES" value="10K"/>
 </parts>
 <sheets>
@@
 <text x="100.584" y="52.07" size="1.778" layer="91">ADR: 100</text>
 <text x="12.7" y="60.96" size="1.778" layer="91" rot="R90">Fan Connectors</text>
+<text x="127" y="10.16" size="1.778" layer="91">Screws</text>
 </plain>
 <instances>
@@
 <instance part="C16" gate="G$1" x="76.2" y="58.42"/>
 <instance part="C17" gate="G$1" x="76.2" y="38.1"/>
-<instance part="JP4" gate="G$1" x="17.78" y="81.28"/>
+<instance part="JP4" gate="G$1" x="17.78" y="83.82"/>
 <instance part="JP5" gate="G$1" x="17.78" y="63.5"/>
 <instance part="JP6" gate="G$1" x="226.06" y="142.24"/>
@@
 <instance part="JP14" gate="G$1" x="7.62" y="33.02"/>
 <instance part="JP15" gate="G$1" x="25.4" y="33.02"/>
+<instance part="U18" gate="G$1" x="43.18" y="83.82" rot="R180"/>
+<instance part="U19" gate="G$1" x="43.18" y="63.5" rot="R180"/>
+<instance part="R3" gate="G$1" x="33.02" y="76.2" rot="R180"/>
+<instance part="R5" gate="G$1" x="33.02" y="55.88" rot="R180"/>
 </instances>
 <busses>
@@
 </segment>
 <segment>
-<pinref part="JP5" gate="G$1" pin="1"/>
-<wire x1="25.4" y1="60.96" x2="30.48" y2="60.96" width="0.2032" layer="91"/>
-<label x="25.4" y="60.96" size="1.778" layer="95"/>
-</segment>
-<segment>
-<pinref part="JP4" gate="G$1" pin="1"/>
-<wire x1="25.4" y1="78.74" x2="30.48" y2="78.74" width="0.2032" layer="91"/>
-<label x="25.4" y="78.74" size="1.778" layer="95"/>
-</segment>
-<segment>
 <pinref part="JP14" gate="G$1" pin="1"/>
 <wire x1="15.24" y1="33.02" x2="20.32" y2="33.02" width="0.2032" layer="91"/>
 <label x="15.24" y="33.02" size="1.778" layer="95"/>
+</segment>
+<segment>
+<pinref part="U19" gate="G$1" pin="S"/>
+<wire x1="33.02" y1="66.04" x2="27.94" y2="66.04" width="0.2032" layer="91"/>
+<label x="27.94" y="66.04" size="1.778" layer="95"/>
+</segment>
+<segment>
+<pinref part="U18" gate="G$1" pin="S"/>
+<wire x1="33.02" y1="86.36" x2="27.94" y2="86.36" width="0.2032" layer="91"/>
+<label x="27.94" y="86.36" size="1.778" layer="95"/>
+</segment>
+<segment>
+<pinref part="R3" gate="G$1" pin="1"/>
+<wire x1="38.1" y1="76.2" x2="43.18" y2="76.2" width="0.2032" layer="91"/>
+<label x="38.1" y="76.2" size="1.778" layer="95"/>
+</segment>
+<segment>
+<pinref part="R5" gate="G$1" pin="1"/>
+<wire x1="38.1" y1="55.88" x2="43.18" y2="55.88" width="0.2032" layer="91"/>
+<label x="38.1" y="55.88" size="1.778" layer="95"/>
 </segment>
 </net>
@@
 <segment>
 <pinref part="JP4" gate="G$1" pin="2"/>
-<wire x1="25.4" y1="81.28" x2="30.48" y2="81.28" width="0.2032" layer="91"/>
-<label x="25.4" y="81.28" size="1.778" layer="95"/>
+<wire x1="25.4" y1="83.82" x2="30.48" y2="83.82" width="0.2032" layer="91"/>
+<label x="25.4" y="83.82" size="1.778" layer="95"/>
 </segment>
 <segment>
@@
 </segment>
 </net>
+<net name="N$1" class="0">
+<segment>
+<pinref part="JP5" gate="G$1" pin="1"/>
+<wire x1="25.4" y1="60.96" x2="27.94" y2="60.96" width="0.2032" layer="91"/>
+<pinref part="U19" gate="G$1" pin="D"/>
+<pinref part="R5" gate="G$1" pin="2"/>
+<wire x1="27.94" y1="60.96" x2="33.02" y2="60.96" width="0.2032" layer="91"/>
+<wire x1="27.94" y1="55.88" x2="27.94" y2="60.96" width="0.2032" layer="91"/>
+</segment>
+</net>
+<net name="N$15" class="0">
+<segment>
+<pinref part="JP4" gate="G$1" pin="1"/>
+<wire x1="25.4" y1="81.28" x2="27.94" y2="81.28" width="0.2032" layer="91"/>
+<pinref part="U18" gate="G$1" pin="D"/>
+<pinref part="R3" gate="G$1" pin="2"/>
+<wire x1="27.94" y1="81.28" x2="33.02" y2="81.28" width="0.2032" layer="91"/>
+<wire x1="27.94" y1="76.2" x2="27.94" y2="81.28" width="0.2032" layer="91"/>
+</segment>
+</net>
+<net name="FAN2" class="0">
+<segment>
+<pinref part="U19" gate="G$1" pin="G"/>
+<wire x1="50.8" y1="63.5" x2="55.88" y2="63.5" width="0.2032" layer="91"/>
+<label x="50.8" y="63.5" size="1.778" layer="95"/>
+</segment>
+</net>
+<net name="FAN1" class="0">
+<segment>
+<pinref part="U18" gate="G$1" pin="G"/>
+<wire x1="50.8" y1="83.82" x2="55.88" y2="83.82" width="0.2032" layer="91"/>
+<label x="50.8" y="83.82" size="1.778" layer="95"/>
+</segment>
+</net>

Commit message: FishLight_PCB: Added Red and Green labels
Added Red and Green text labels to the extra CAT4101s.
Other:
- note added: "GRN"
- note added: "RD"
Changed lines of the file:
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@@
 <text x="12.7" y="60.96" size="1.778" layer="91" rot="R90">Fan Connectors</text>
 <text x="127" y="10.16" size="1.778" layer="91">Screws</text>
+<text x="172.72" y="180.34" size="1.778" layer="91">RD</text>
+<text x="170.18" y="165.1" size="1.778" layer="91">GRN</text>
 </plain>
 <instances>

Commit message: FishLight_PCB: Fixed fan transistors
Fixed the fan connector transistor pull down resistors.  These were
connected to drain but they need to be connected to gate so that the
transistor shuts off correctly.  Also added some Solid State Relays to
possibly turn on and off some AC loads (such as a pump or the heater)
for emergency situations.  These will probably go away though.  Kind of
an interesting idea is all.
Parts:
- added R11, R12: 10K, SparkFun-Resistors:RESISTOR0603-RES
- added U20, U21: RELAY-SOLIDSTATEPTH, SparkFun-Electromechanical:RELAY-SOLIDSTATEPTH
- R1, R2: value 10K -> 4.7K
Connections:
- new net N$16: R11.1, U19.D
- new net N$18: JP5.1, R11.2
- net FAN1: now also R3.2
- net FAN2: now also R5.2
- net N$1: now also JP4.1, R12.2; no longer JP5.1, R5.2, U19.D
- net N$15: now also R12.1; no longer JP4.1, R3.2
Other:
- note added: "I-Limit"
- moved on the sheet: JP4, JP5, R3, R5
Changed lines of the file:
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@@
 <part name="C4" library="SparkFun-Capacitors" deviceset="0.1UF-25V(+80/-20%)(0603)" device="" value="0.1uF"/>
 <part name="C5" library="SparkFun-Capacitors" deviceset="0.1UF-25V(+80/-20%)(0603)" device="" value="0.1uF"/>
-<part name="R1" library="SparkFun-Resistors" deviceset="RESISTOR" device="0603" value="10K"/>
-<part name="R2" library="SparkFun-Resistors" deviceset="RESISTOR" device="0603" value="10K"/>
+<part name="R1" library="SparkFun-Resistors" deviceset="RESISTOR" device="0603" value="4.7K"/>
+<part name="R2" library="SparkFun-Resistors" deviceset="RESISTOR" device="0603" value="4.7K"/>
 <part name="5V1" library="SparkFun-Aesthetics" deviceset="5V" device=""/>
 <part name="C7" library="SparkFun-Capacitors" deviceset="0.1UF-25V(+80/-20%)(0603)" device="" value="0.1uF"/>
@@
 <part name="R3" library="SparkFun-Resistors" deviceset="RESISTOR" device="0603-RES" value="10K"/>
 <part name="R5" library="SparkFun-Resistors" deviceset="RESISTOR" device="0603-RES" value="10K"/>
+<part name="U20" library="SparkFun-Electromechanical" deviceset="RELAY-SOLIDSTATE" device="PTH"/>
+<part name="U21" library="SparkFun-Electromechanical" deviceset="RELAY-SOLIDSTATE" device="PTH"/>
+<part name="R11" library="SparkFun-Resistors" deviceset="RESISTOR" device="0603-RES" value="10K"/>
+<part name="R12" library="SparkFun-Resistors" deviceset="RESISTOR" device="0603-RES" value="10K"/>
 </parts>
 <sheets>
@@
 <text x="100.584" y="72.39" size="1.778" layer="91">ADR: 11</text>
 <text x="100.584" y="52.07" size="1.778" layer="91">ADR: 100</text>
-<text x="12.7" y="60.96" size="1.778" layer="91" rot="R90">Fan Connectors</text>
+<text x="5.08" y="60.96" size="1.778" layer="91" rot="R90">Fan Connectors</text>
 <text x="127" y="10.16" size="1.778" layer="91">Screws</text>
 <text x="172.72" y="180.34" size="1.778" layer="91">RD</text>
 <text x="170.18" y="165.1" size="1.778" layer="91">GRN</text>
+<text x="22.86" y="55.88" size="1.778" layer="91">I-Limit</text>
+<text x="22.86" y="76.2" size="1.778" layer="91">I-Limit</text>
 </plain>
 <instances>
@@
 <instance part="C16" gate="G$1" x="76.2" y="58.42"/>
 <instance part="C17" gate="G$1" x="76.2" y="38.1"/>
-<instance part="JP4" gate="G$1" x="17.78" y="83.82"/>
-<instance part="JP5" gate="G$1" x="17.78" y="63.5"/>
+<instance part="JP4" gate="G$1" x="10.16" y="83.82"/>
+<instance part="JP5" gate="G$1" x="10.16" y="63.5"/>
 <instance part="JP6" gate="G$1" x="226.06" y="142.24"/>
 <instance part="JP7" gate="G$1" x="215.9" y="144.78" rot="R180"/>
@@
 <instance part="U18" gate="G$1" x="43.18" y="83.82" rot="R180"/>
 <instance part="U19" gate="G$1" x="43.18" y="63.5" rot="R180"/>
-<instance part="R3" gate="G$1" x="33.02" y="76.2" rot="R180"/>
-<instance part="R5" gate="G$1" x="33.02" y="55.88" rot="R180"/>
+<instance part="R3" gate="G$1" x="55.88" y="78.74" rot="R90"/>
+<instance part="R5" gate="G$1" x="55.88" y="58.42" rot="R90"/>
+<instance part="U20" gate="G$1" x="144.78" y="63.5"/>
+<instance part="U21" gate="G$1" x="144.78" y="48.26"/>
+<instance part="R11" gate="G$1" x="25.4" y="60.96" rot="R180"/>
+<instance part="R12" gate="G$1" x="25.4" y="81.28" rot="R180"/>
 </instances>
 <busses>
@@
 <segment>
 <pinref part="R3" gate="G$1" pin="1"/>
-<wire x1="38.1" y1="76.2" x2="43.18" y2="76.2" width="0.2032" layer="91"/>
-<label x="38.1" y="76.2" size="1.778" layer="95"/>
+<wire x1="55.88" y1="73.66" x2="55.88" y2="68.58" width="0.2032" layer="91"/>
+<label x="55.88" y="68.58" size="1.778" layer="95" rot="R90"/>
 </segment>
 <segment>
 <pinref part="R5" gate="G$1" pin="1"/>
-<wire x1="38.1" y1="55.88" x2="43.18" y2="55.88" width="0.2032" layer="91"/>
-<label x="38.1" y="55.88" size="1.778" layer="95"/>
+<wire x1="55.88" y1="53.34" x2="55.88" y2="48.26" width="0.2032" layer="91"/>
+<label x="55.88" y="48.26" size="1.778" layer="95" rot="R90"/>
 </segment>
 </net>
@@
 <segment>
 <pinref part="JP4" gate="G$1" pin="2"/>
-<wire x1="25.4" y1="83.82" x2="30.48" y2="83.82" width="0.2032" layer="91"/>
-<label x="25.4" y="83.82" size="1.778" layer="95"/>
+<wire x1="17.78" y1="83.82" x2="22.86" y2="83.82" width="0.2032" layer="91"/>
+<label x="17.78" y="83.82" size="1.778" layer="95"/>
 </segment>
 <segment>
 <pinref part="JP5" gate="G$1" pin="2"/>
-<wire x1="25.4" y1="63.5" x2="30.48" y2="63.5" width="0.2032" layer="91"/>
-<label x="25.4" y="63.5" size="1.778" layer="95"/>
+<wire x1="17.78" y1="63.5" x2="22.86" y2="63.5" width="0.2032" layer="91"/>
+<label x="17.78" y="63.5" size="1.778" layer="95"/>
 </segment>
 <segment>
@@
 </segment>
 </net>
-<net name="N$1" class="0">
-<segment>
-<pinref part="JP5" gate="G$1" pin="1"/>
-<wire x1="25.4" y1="60.96" x2="27.94" y2="60.96" width="0.2032" layer="91"/>
-<pinref part="U19" gate="G$1" pin="D"/>
-<pinref part="R5" gate="G$1" pin="2"/>
-<wire x1="27.94" y1="60.96" x2="33.02" y2="60.96" width="0.2032" layer="91"/>
-<wire x1="27.94" y1="55.88" x2="27.94" y2="60.96" width="0.2032" layer="91"/>
-</segment>
-</net>
-<net name="N$15" class="0">
-<segment>
-<pinref part="JP4" gate="G$1" pin="1"/>
-<wire x1="25.4" y1="81.28" x2="27.94" y2="81.28" width="0.2032" layer="91"/>
-<pinref part="U18" gate="G$1" pin="D"/>
-<pinref part="R3" gate="G$1" pin="2"/>
-<wire x1="27.94" y1="81.28" x2="33.02" y2="81.28" width="0.2032" layer="91"/>
-<wire x1="27.94" y1="76.2" x2="27.94" y2="81.28" width="0.2032" layer="91"/>
-</segment>
-</net>
 <net name="FAN2" class="0">
 <segment>
@@
 <wire x1="50.8" y1="63.5" x2="55.88" y2="63.5" width="0.2032" layer="91"/>
 <label x="50.8" y="63.5" size="1.778" layer="95"/>
+<pinref part="R5" gate="G$1" pin="2"/>
+<wire x1="55.88" y1="63.5" x2="58.42" y2="63.5" width="0.2032" layer="91"/>
 </segment>
 </net>
@@
 <wire x1="50.8" y1="83.82" x2="55.88" y2="83.82" width="0.2032" layer="91"/>
 <label x="50.8" y="83.82" size="1.778" layer="95"/>
-</segment>
-</net>
+<pinref part="R3" gate="G$1" pin="2"/>
+<wire x1="55.88" y1="83.82" x2="58.42" y2="83.82" width="0.2032" layer="91"/>
+</segment>
+</net>
+<net name="N$1" class="0">
+<segment>
+<pinref part="JP4" gate="G$1" pin="1"/>
+<pinref part="R12" gate="G$1" pin="2"/>
+<wire x1="17.78" y1="81.28" x2="20.32" y2="81.28" width="0.2032" layer="91"/>
+</segment>
+</net>
+<net name="N$15" class="0">
+<segment>
+<pinref part="R12" gate="G$1" pin="1"/>
+<pinref part="U18" gate="G$1" pin="D"/>
+<wire x1="30.48" y1="81.28" x2="33.02" y2="81.28" width="0.2032" layer="91"/>
+</segment>
+</net>
+<net name="N$16" class="0">
+<segment>
+<pinref part="U19" gate="G$1" pin="D"/>
+<pinref part="R11" gate="G$1" pin="1"/>
+<wire x1="33.02" y1="60.96" x2="30.48" y2="60.96" width="0.2032" layer="91"/>
+</segment>
+</net>
+<net name="N$18" class="0">
+<segment>
+<pinref part="R11" gate="G$1" pin="2"/>
+<pinref part="JP5" gate="G$1" pin="1"/>
+<wire x1="20.32" y1="60.96" x2="17.78" y2="60.96" width="0.2032" layer="91"/>
+</segment>
+</net>

Commit message: FishLight_PCB: Added LED strings 4 - 8
Added LED strings 4 - 8 and removed the 'green' string.  This will allow
me to control 2 tanks or one really big tank in the future.  Added all
of the accompanying parts and moved a lot of stuff around to make it all
fit on the schematic.  Still need to lay them out on the board tho.
Parts:
- added C18, C19, C20, C21, C22, C23, C24: 0.1uF, SparkFun-Capacitors:0.1UF-25V(+80/-20%)(0603)
- added JP16, JP20: (no value), Mikes-Stuff:M03SCREW
- added R13, R14, R15: (no value), SparkFun-Resistors:RESISTOR2010
- added U22: AD5248MSOP-10, Mikes-Stuff:AD5248MSOP-10
- added U23, U24, U25: CAT4101TO-263, Mikes-Stuff:CAT4101TO-263
- added U26, U27, U28: INA219SOT23-8, Mikes-Stuff:INA219SOT23-8
Connections:
- removed net N$14: U10.B1
- removed net N$17: U10.B2
- removed net N$3: JP11.3
- removed net N$6: JP10.1
- new net LED6: JP11.3, R13.1, U26.V-
- new net LED7: JP20.1, R14.1, U27.V-
- new net LED8: JP20.2, R15.1, U28.V-
- new net LG6: JP10.1, U23.LED
- new net LG7: JP16.3, U25.LED
- new net LG8: JP16.2, U24.LED
- new net LR6: U10.W1, U23.RSET
- new net LR7: U22.W2, U25.RSET
- new net LR8: U22.W1, U24.RSET
- new net N$22: JP20.3
- new net N$27: JP16.1
- net 24V: now also R13.2, R14.2, R15.2, U26.V+, U27.V+, U28.V+
- net 5V: now also C18.2, C19.1, C20.1, C21.1, C22.2, C23.2, C24.2, U12.A0, U22.AD0, U22.AD1, U22.VDD, U23.VIN, U24.VIN, U25.VIN, U26.A0, U26.A1, U26.VDD, U27.A1, U27.VDD, U28.A1, U28.VDD
- net D0: now also U7.PWM
- net D1: now also U23.PWM
- net D2: now also U25.PWM
- net D3: now also U24.PWM
- net D4: no longer U7.PWM
- net GND: now also C18.1, C19.2, C20.2, C21.2, C22.1, C23.1, C24.1, U10.B1, U10.B2, U11.A0, U11.A1, U12.A1, U13.A1, U22.B1, U22.B2, U22.GND, U23.GND, U24.GND, U25.GND, U26.GND, U27.GND, U28.GND
- net SCL: now also U11.SCL, U12.SCL, U13.SCL, U22.SCL, U26.SCL, U27.SCL, U28.A0, U28.SCL
- net SDA: now also U11.SDA, U12.SDA, U13.A0, U13.SDA, U22.SDA, U26.SDA, U27.A0, U27.SDA, U28.SDA
Other:
- note added: "ADR: 101"
- note added: "ADR: 110"
- note added: "ADR: 111"
- note added: "BL2"
- note added: "CW2"
- note added: "RD2"
- note added: "WW2"
- note removed: "GRN"
- moved on the sheet: C1, C10, C11, C13, C16, C17, C2, C3, C4, C5, C7, C8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
