File: FishLight-v01.sch (EAGLE design)
At the start: 90 parts, among them U1 SPARK_CORECORE, U10 AD5248MSOP-10, U11 INA219SOT23-8, U12 INA219SOT23-8, U13 INA219SOT23-8, U14 INA219SOT23-8, U15 INA219SOT23-8, U16 UA7812D2PAK-3, U17 L7805D2PAK-2, U18 RK7002BSOT23-3, U19 RK7002BSOT23-3, U2 RTCBREAKOUT, U20 RELAY-SOLIDSTATEPTH, U21 RELAY-SOLIDSTATEPTH, U22 AD5248MSOP-10, U23 CAT4101TO-263, U24 CAT4101TO-263, U25 CAT4101TO-263, U26 INA219SOT23-8, U27 INA219SOT23-8, U28 INA219SOT23-8, U3 CAT4101TO-263, U4 CAT4101TO-263, U5 CAT4101TO-263, U6 CAT4101TO-263, U7 CAT4101TO-263, U8 AD5248MSOP-10, U9 AD5248MSOP-10

Commit message: FishLight_PCB: Replaced the RTC and added VIAs
Replaced the giant RTC breakout board with the new DS3231M RTC.  This
can fit right under the Spark Core so it takes up very little space.
The battery is still kinda big but its not a big deal.  Also added VIAs
to the CAT4101s that are on the top side and to the I-Sense resistors
that are new.
Parts:
- removed U2: RTCBREAKOUT, Mikes-Stuff:RTCBREAKOUT
- added BAT1: (no value), SparkFun-Electromechanical:BATTERY12PTH
- added C25: 0.1uF, SparkFun-Capacitors:0.1UF-25V(+80/-20%)(0603)
- added U29: DS3231MSOIC-8, Mikes-Stuff:DS3231MSOIC-8
Connections:
- removed net N$22: JP20.3
- removed net N$27: JP16.1
- new net N$3: BAT1.+, U29.VBAT
- net 5V: now also C25.1, U29.VCC; no longer U2.5V
- net GND: now also BAT1.-, C25.2, U29.GND; no longer U2.GND
- net LED7: now also JP20.2; no longer JP20.1
- net LED8: now also JP20.3; no longer JP20.2
- net LG7: now also JP16.2; no longer JP16.3
- net LG8: now also JP16.1; no longer JP16.2
- net SCL: now also U29.SCL; no longer U2.SCL
- net SDA: now also U29.SDA; no longer U2.SDA
- net SQW: now also U29.SQW; no longer U2.SQW
Other:
- moved on the sheet: R1, R2
Changed lines of the file:
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@@
 <part name="STANDOFF4" library="SparkFun-Electromechanical" deviceset="STAND-OFF" device=""/>
 <part name="FRAME1" library="SparkFun-Aesthetics" deviceset="FRAME-LETTER" device=""/>
-<part name="U2" library="Mikes-Stuff" deviceset="RTCBREAKOUT" device=""/>
 <part name="U3" library="Mikes-Stuff" deviceset="CAT4101" device="TO-263"/>
 <part name="U4" library="Mikes-Stuff" deviceset="CAT4101" device="TO-263"/>
@@
 <part name="C23" library="SparkFun-Capacitors" deviceset="0.1UF-25V(+80/-20%)(0603)" device="" value="0.1uF"/>
 <part name="C24" library="SparkFun-Capacitors" deviceset="0.1UF-25V(+80/-20%)(0603)" device="" value="0.1uF"/>
+<part name="U29" library="Mikes-Stuff" deviceset="DS3231M" device="SOIC-8"/>
+<part name="BAT1" library="SparkFun-Electromechanical" deviceset="BATTERY" device="12PTH"/>
+<part name="C25" library="SparkFun-Capacitors" deviceset="0.1UF-25V(+80/-20%)(0603)" device="" value="0.1uF"/>
 </parts>
 <sheets>
@@
 <text x="124.46" y="182.88" size="1.778" layer="91">WW</text>
 <text x="172.72" y="182.88" size="1.778" layer="91">BL</text>
-<text x="220.98" y="60.96" size="1.778" layer="91" rot="R90">External TMP Sensors</text>
+<text x="223.52" y="58.42" size="1.778" layer="91" rot="R90">External TMP Sensors</text>
 <text x="220.98" y="132.08" size="1.778" layer="91" rot="R90">Screw Terminals</text>
 <text x="111.76" y="121.92" size="1.778" layer="91" rot="R180">I-sense</text>
@@
 <instance part="FRAME1" gate="G$1" x="0" y="0"/>
 <instance part="FRAME1" gate="G$2" x="147.32" y="0"/>
-<instance part="U2" gate="RTC" x="228.6" y="45.72"/>
 <instance part="U3" gate="G$1" x="119.38" y="177.8"/>
 <instance part="U4" gate="G$1" x="167.64" y="177.8"/>
@@
 <instance part="C4" gate="G$1" x="187.96" y="160.02"/>
 <instance part="C5" gate="G$1" x="139.7" y="144.78"/>
-<instance part="R1" gate="G$1" x="208.28" y="53.34" rot="R90"/>
-<instance part="R2" gate="G$1" x="203.2" y="53.34" rot="R90"/>
-<instance part="5V1" gate="G$1" x="205.74" y="58.42"/>
+<instance part="R1" gate="G$1" x="241.3" y="45.72"/>
+<instance part="R2" gate="G$1" x="241.3" y="50.8"/>
+<instance part="5V1" gate="G$1" x="246.38" y="48.26" rot="R270"/>
 <instance part="C7" gate="G$1" x="157.48" y="106.68"/>
 <instance part="C8" gate="G$1" x="157.48" y="86.36"/>
@@
 <instance part="C23" gate="G$1" x="63.5" y="66.04"/>
 <instance part="C24" gate="G$1" x="63.5" y="45.72"/>
+<instance part="U29" gate="G$1" x="218.44" y="45.72"/>
+<instance part="BAT1" gate="G$1" x="241.3" y="38.1" rot="R270"/>
+<instance part="C25" gate="G$1" x="215.9" y="55.88" rot="R90"/>
 </instances>
 <busses>
@@
 </segment>
 <segment>
-<wire x1="215.9" y1="48.26" x2="208.28" y2="48.26" width="0.1524" layer="91"/>
-<label x="210.82" y="48.26" size="1.778" layer="95"/>
-<pinref part="U2" gate="RTC" pin="SDA"/>
+<wire x1="231.14" y1="45.72" x2="236.22" y2="45.72" width="0.1524" layer="91"/>
+<label x="231.14" y="45.72" size="1.778" layer="95"/>
 <pinref part="R1" gate="G$1" pin="1"/>
+<pinref part="U29" gate="G$1" pin="SDA"/>
 </segment>
 <segment>
@@
 </segment>
 <segment>
-<wire x1="215.9" y1="45.72" x2="208.28" y2="45.72" width="0.1524" layer="91"/>
-<label x="210.82" y="45.72" size="1.778" layer="95"/>
-<pinref part="U2" gate="RTC" pin="SCL"/>
+<wire x1="231.14" y1="48.26" x2="236.22" y2="48.26" width="0.1524" layer="91"/>
+<label x="231.14" y="48.26" size="1.778" layer="95"/>
 <pinref part="R2" gate="G$1" pin="1"/>
-<wire x1="208.28" y1="45.72" x2="203.2" y2="45.72" width="0.2032" layer="91"/>
-<wire x1="203.2" y1="45.72" x2="203.2" y2="48.26" width="0.2032" layer="91"/>
+<wire x1="236.22" y1="50.8" x2="236.22" y2="48.26" width="0.2032" layer="91"/>
+<pinref part="U29" gate="G$1" pin="SCL"/>
 </segment>
 <segment>
@@
 </segment>
 <segment>
-<wire x1="241.3" y1="48.26" x2="246.38" y2="48.26" width="0.1524" layer="91"/>
-<label x="241.3" y="48.26" size="1.778" layer="95"/>
-<pinref part="U2" gate="RTC" pin="GND"/>
+<wire x1="231.14" y1="40.64" x2="236.22" y2="40.64" width="0.1524" layer="91"/>
+<label x="231.14" y="40.64" size="1.778" layer="95"/>
+<pinref part="BAT1" gate="G$1" pin="-"/>
+<wire x1="241.3" y1="33.02" x2="236.22" y2="33.02" width="0.2032" layer="91"/>
+<wire x1="236.22" y1="33.02" x2="236.22" y2="40.64" width="0.2032" layer="91"/>
+<pinref part="U29" gate="G$1" pin="GND"/>
 </segment>
 <segment>
@@
 <label x="116.84" y="109.22" size="1.778" layer="95"/>
 </segment>
+<segment>
+<pinref part="C25" gate="G$1" pin="2"/>
+<wire x1="218.44" y1="55.88" x2="223.52" y2="55.88" width="0.2032" layer="91"/>
+<label x="218.44" y="55.88" size="1.778" layer="95"/>
+</segment>
 </net>
 <net name="5V" class="0">
@@
 </segment>
 <segment>
-<wire x1="241.3" y1="43.18" x2="246.38" y2="43.18" width="0.1524" layer="91"/>
-<label x="241.3" y="43.18" size="1.778" layer="95"/>
-<pinref part="U2" gate="RTC" pin="5V"/>
+<wire x1="200.66" y1="45.72" x2="205.74" y2="45.72" width="0.1524" layer="91"/>
+<label x="200.66" y="45.72" size="1.778" layer="95"/>
+<pinref part="U29" gate="G$1" pin="VCC"/>
 </segment>
 <segment>
@@
 <wire x1="187.96" y1="165.1" x2="180.34" y2="165.1" width="0.2032" layer="91"/>
 <label x="182.88" y="165.1" size="1.778" layer="95"/>
-</segment>
-<segment>
-<pinref part="R2" gate="G$1" pin="2"/>
-<pinref part="R1" gate="G$1" pin="2"/>
-<wire x1="203.2" y1="58.42" x2="205.74" y2="58.42" width="0.2032" layer="91"/>
-<pinref part="5V1" gate="G$1" pin="5V"/>
-<wire x1="205.74" y1="58.42" x2="208.28" y2="58.42" width="0.2032" layer="91"/>
-<junction x="205.74" y="58.42"/>
 </segment>
 <segment>
@@
 <label x="101.6" y="53.34" size="1.778" layer="95"/>
 </segment>
+<segment>
+<pinref part="R2" gate="G$1" pin="2"/>
+<pinref part="5V1" gate="G$1" pin="5V"/>
+<pinref part="R1" gate="G$1" pin="2"/>
+<wire x1="246.38" y1="50.8" x2="246.38" y2="48.26" width="0.2032" layer="91"/>
+<wire x1="246.38" y1="48.26" x2="246.38" y2="45.72" width="0.2032" layer="91"/>
+</segment>
+<segment>
+<pinref part="C25" gate="G$1" pin="1"/>
+<wire x1="210.82" y1="55.88" x2="205.74" y2="55.88" width="0.2032" layer="91"/>
+<label x="205.74" y="55.88" size="1.778" layer="95"/>
+</segment>
 </net>
 <net name="SQW" class="0">
 <segment>
-<wire x1="215.9" y1="43.18" x2="210.82" y2="43.18" width="0.1524" layer="91"/>
-<label x="210.82" y="43.18" size="1.778" layer="95"/>
-<pinref part="U2" gate="RTC" pin="SQW"/>
+<wire x1="205.74" y1="43.18" x2="200.66" y2="43.18" width="0.1524" layer="91"/>
+<label x="200.66" y="43.18" size="1.778" layer="95"/>
+<pinref part="U29" gate="G$1" pin="SQW"/>
 </segment>
 </net>
@@
 <net name="LED7" class="0">
 <segment>
-<pinref part="JP20" gate="G$1" pin="1"/>
-<wire x1="208.28" y1="147.32" x2="203.2" y2="147.32" width="0.2032" layer="91"/>
-<label x="203.2" y="147.32" size="1.778" layer="95"/>
-</segment>
-<segment>
 <pinref part="U27" gate="G$1" pin="V-"/>
 <pinref part="R14" gate="G$1" pin="1"/>
@@
 <label x="71.12" y="71.12" size="1.778" layer="95"/>
 </segment>
-</net>
-<net name="LED8" class="0">
 <segment>
 <pinref part="JP20" gate="G$1" pin="2"/>
@@
 <label x="203.2" y="144.78" size="1.778" layer="95"/>
 </segment>
+</net>
+<net name="LED8" class="0">
 <segment>
 <pinref part="U28" gate="G$1" pin="V-"/>
@@
 <label x="71.12" y="50.8" size="1.778" layer="95"/>
 </segment>
-</net>
-<net name="N$22" class="0">
 <segment>
 <pinref part="JP20" gate="G$1" pin="3"/>
 <wire x1="208.28" y1="142.24" x2="203.2" y2="142.24" width="0.2032" layer="91"/>
-</segment>
-</net>
-<net name="N$27" class="0">
+<label x="203.2" y="142.24" size="1.778" layer="95"/>
+</segment>
+</net>
+<net name="LG8" class="0">
+<segment>
+<pinref part="U24" gate="G$1" pin="LED"/>
+<wire x1="154.94" y1="129.54" x2="149.86" y2="129.54" width="0.2032" layer="91"/>
+<label x="149.86" y="129.54" size="1.778" layer="95"/>
+</segment>
 <segment>
 <pinref part="JP16" gate="G$1" pin="1"/>
 <wire x1="233.68" y1="142.24" x2="238.76" y2="142.24" width="0.2032" layer="91"/>
-</segment>
-</net>
-<net name="LG8" class="0">
+<label x="233.68" y="142.24" size="1.778" layer="95"/>
+</segment>
+</net>
+<net name="LG7" class="0">
+<segment>
+<pinref part="U25" gate="G$1" pin="LED"/>
+<wire x1="106.68" y1="129.54" x2="101.6" y2="129.54" width="0.2032" layer="91"/>
+<label x="101.6" y="129.54" size="1.778" layer="95"/>
+</segment>
 <segment>
 <pinref part="JP16" gate="G$1" pin="2"/>
@@
 <label x="233.68" y="144.78" size="1.778" layer="95"/>
 </segment>
-<segment>
-<pinref part="U24" gate="G$1" pin="LED"/>
-<wire x1="154.94" y1="129.54" x2="149.86" y2="129.54" width="0.2032" layer="91"/>
-<label x="149.86" y="129.54" size="1.778" layer="95"/>
-</segment>
-</net>
-<net name="LG7" class="0">
-<segment>
-<pinref part="JP16" gate="G$1" pin="3"/>
-<wire x1="233.68" y1="147.32" x2="238.76" y2="147.32" width="0.2032" layer="91"/>
-<label x="233.68" y="147.32" size="1.778" layer="95"/>
-</segment>
-<segment>
-<pinref part="U25" gate="G$1" pin="LED"/>
-<wire x1="106.68" y1="129.54" x2="101.6" y2="129.54" width="0.2032" layer="91"/>
-<label x="101.6" y="129.54" size="1.778" layer="95"/>
-</segment>
-</net>
+</net>
+<net name="N$3" class="0">
+<segment>
+<pinref part="U29" gate="G$1" pin="VBAT"/>
+<pinref part="BAT1" gate="G$1" pin="+"/>
+<wire x1="231.14" y1="43.18" x2="241.3" y2="43.18" width="0.2032" layer="91"/>
+</segment>
+</net>

Commit message: FishLight_PCB: Swapped out the LCD connector
The LCD connector was just a 5pin header.  Now it is a polarized header
so that it cannot be plugged in backwards on accident.  Also moved some
things around to get straighter lines on the I2C bus.
Parts:
- JP18: device SparkFun-Connectors:M05PTH -> Mikes-Stuff:M05POLAR
Changed lines of the file:
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@@
 <grid distance="0.1" unitdist="inch" unit="inch" style="lines" multiple="1" display="no" altdistance="0.01" altunitdist="inch" altunit="inch"/>
 <layers>
-<layer number="1" name="Top" color="4" fill="1" visible="no" active="no"/>
-<layer number="16" name="Bottom" color="1" fill="1" visible="no" active="no"/>
-<layer number="17" name="Pads" color="2" fill="1" visible="no" active="no"/>
-<layer number="18" name="Vias" color="2" fill="1" visible="no" active="no"/>
-<layer number="19" name="Unrouted" color="6" fill="1" visible="no" active="no"/>
-<layer number="20" name="Dimension" color="15" fill="1" visible="no" active="no"/>
-<layer number="21" name="tPlace" color="16" fill="1" visible="no" active="no"/>
-<layer number="22" name="bPlace" color="14" fill="1" visible="no" active="no"/>
-<layer number="23" name="tOrigins" color="15" fill="1" visible="no" active="no"/>
-<layer number="24" name="bOrigins" color="15" fill="1" visible="no" active="no"/>
-<layer number="25" name="tNames" color="7" fill="1" visible="no" active="no"/>
-<layer number="26" name="bNames" color="7" fill="1" visible="no" active="no"/>
-<layer number="27" name="tValues" color="7" fill="1" visible="no" active="no"/>
-<layer number="28" name="bValues" color="7" fill="1" visible="no" active="no"/>
+<layer number="1" name="Top" color="4" fill="1" visible="yes" active="no"/>
+<layer number="16" name="Bottom" color="1" fill="1" visible="yes" active="no"/>
+<layer number="17" name="Pads" color="2" fill="1" visible="yes" active="no"/>
+<layer number="18" name="Vias" color="2" fill="1" visible="yes" active="no"/>
+<layer number="19" name="Unrouted" color="6" fill="1" visible="yes" active="no"/>
+<layer number="20" name="Dimension" color="15" fill="1" visible="yes" active="no"/>
+<layer number="21" name="tPlace" color="16" fill="1" visible="yes" active="no"/>
+<layer number="22" name="bPlace" color="14" fill="1" visible="yes" active="no"/>
+<layer number="23" name="tOrigins" color="15" fill="1" visible="yes" active="no"/>
+<layer number="24" name="bOrigins" color="15" fill="1" visible="yes" active="no"/>
+<layer number="25" name="tNames" color="7" fill="1" visible="yes" active="no"/>
+<layer number="26" name="bNames" color="7" fill="1" visible="yes" active="no"/>
+<layer number="27" name="tValues" color="7" fill="1" visible="yes" active="no"/>
+<layer number="28" name="bValues" color="7" fill="1" visible="yes" active="no"/>
 <layer number="29" name="tStop" color="7" fill="3" visible="no" active="no"/>
 <layer number="30" name="bStop" color="7" fill="6" visible="no" active="no"/>
@@
 <layer number="35" name="tGlue" color="7" fill="4" visible="no" active="no"/>
 <layer number="36" name="bGlue" color="7" fill="5" visible="no" active="no"/>
-<layer number="37" name="tTest" color="7" fill="1" visible="no" active="no"/>
-<layer number="38" name="bTest" color="7" fill="1" visible="no" active="no"/>
+<layer number="37" name="tTest" color="7" fill="1" visible="yes" active="no"/>
+<layer number="38" name="bTest" color="7" fill="1" visible="yes" active="no"/>
 <layer number="39" name="tKeepout" color="4" fill="11" visible="no" active="no"/>
 <layer number="40" name="bKeepout" color="1" fill="11" visible="no" active="no"/>
@@
 <layer number="44" name="Drills" color="7" fill="1" visible="no" active="no"/>
 <layer number="45" name="Holes" color="7" fill="1" visible="no" active="no"/>
-<layer number="46" name="Milling" color="3" fill="1" visible="no" active="no"/>
-<layer number="47" name="Measures" color="7" fill="1" visible="no" active="no"/>
-<layer number="48" name="Document" color="7" fill="1" visible="no" active="no"/>
-<layer number="49" name="Reference" color="7" fill="1" visible="no" active="no"/>
-<layer number="50" name="dxf" color="7" fill="1" visible="no" active="no"/>
-<layer number="51" name="tDocu" color="6" fill="1" visible="no" active="no"/>
-<layer number="52" name="bDocu" color="5" fill="1" visible="no" active="no"/>
-<layer number="53" name="tGND_GNDA" color="7" fill="9" visible="no" active="no"/>
-<layer number="54" name="bGND_GNDA" color="1" fill="9" visible="no" active="no"/>
-<layer number="56" name="wert" color="7" fill="1" visible="no" active="no"/>
+<layer number="46" name="Milling" color="3" fill="1" visible="yes" active="no"/>
+<layer number="47" name="Measures" color="7" fill="1" visible="yes" active="no"/>
+<layer number="48" name="Document" color="7" fill="1" visible="yes" active="no"/>
+<layer number="49" name="Reference" color="7" fill="1" visible="yes" active="no"/>
+<layer number="50" name="dxf" color="7" fill="1" visible="yes" active="no"/>
+<layer number="51" name="tDocu" color="6" fill="1" visible="yes" active="no"/>
+<layer number="52" name="bDocu" color="5" fill="1" visible="yes" active="no"/>
+<layer number="53" name="tGND_GNDA" color="7" fill="9" visible="yes" active="no"/>
+<layer number="54" name="bGND_GNDA" color="1" fill="9" visible="yes" active="no"/>
+<layer number="56" name="wert" color="7" fill="1" visible="yes" active="no"/>
 <layer number="91" name="Nets" color="2" fill="1" visible="yes" active="yes"/>
 <layer number="92" name="Busses" color="1" fill="1" visible="yes" active="yes"/>
@@
 <part name="U1" library="Spark" deviceset="SPARK_CORE" device="CORE"/>
 <part name="R4" library="SparkFun-Resistors" deviceset="RESISTOR" device="0603-RES" value="4.7K"/>
-<part name="JP18" library="SparkFun-Connectors" deviceset="M05" device="PTH"/>
+<part name="JP18" library="Mikes-Stuff" deviceset="M05" device="POLAR"/>
 <part name="R6" library="SparkFun-Resistors" deviceset="RESISTOR" device="2010"/>
 <part name="R7" library="SparkFun-Resistors" deviceset="RESISTOR" device="2010"/>

Commit message: FishLight_PCB: Shrink schematic symbols
In an effort to save space, I have shrunk many of my own schematic
symbols by making pins small instead of medium in their properties.
This saved a lot of space in the schematic.  I also added 9 2pin screw
terminals for 12V devices and changed the current limiting resistor on
the fans to limit current to the transistor, not the fan itself.  I may
also put some LEDs on the 12V devices and the SSRs in order to show what
devices are on or off.  May also want to add another SSR.
Parts:
- added JP17, JP19, JP21, JP22, JP23, JP24, JP25, JP26, JP27: M023.5MM, SparkFun-Connectors:M023.5MM
- R11, R12: value 10K -> 330; device SparkFun-Resistors:RESISTOR0603-RES -> SparkFun-Resistors:RESISTOR0603
Connections:
- new net N$17: JP21.1, JP26.1
- new net N$21: JP24.1, JP27.1
- new net N$23: JP23.1
- new net N$25: JP22.1
- new net N$27: JP17.1
- new net N$29: JP25.1
- new net N$6: JP19.1
- net FAN1: now also R11.2; no longer U18.G
- net FAN2: now also R12.2; no longer U19.G
- net GND: now also JP17.2, JP19.2, JP21.2, JP22.2, JP23.2, JP24.2, JP25.2, JP26.2, JP27.2
- net N$1: now also U18.D; no longer R12.2
- net N$15: now also JP5.1, U19.D; no longer R12.1, U18.D
- net N$16: now also U18.G; no longer U19.D
- net N$18: now also R12.1, U19.G; no longer JP5.1, R11.2
Other:
- note removed: "I-Limit"
- moved on the sheet: BAT1, C1, C10, C11, C12, C13, C14, C15, C16, C17, C18, C19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

Commit message: FishLight_PCB: Add second SCH frame and replace 12V reg
Added a second Schematic frame and placed it in a place that will allow
it to be printed correctly.  This will open up a lot of room for more
devices on my schematic, specifically my 12V devices.  Also changed my
12V regulator to a higher current (3A) version.  This will allow me to
have more 12V devices.  Also added 3 more, total 5, SSRs.  This may be
too many for my case but it will be interesting to try it out.
Parts:
- added FRAME2: FRAME-LETTER, SparkFun-Aesthetics:FRAME-LETTER
- added U2, U30, U31: RELAY-SOLIDSTATEPTH, SparkFun-Electromechanical:RELAY-SOLIDSTATEPTH
- U16: value UA7812D2PAK-3 -> MIC29300D2PAK-3; device Mikes-Stuff:UA7812D2PAK-3 -> Mikes-Stuff:MIC29300D2PAK-3
Other:
- moved on the sheet: C10, C11, C12, C13, C14, C15, C16, C17, C18, C22, C23, C24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
