File: FishLight-v01.sch (EAGLE design)
At the start: 105 parts, among them U1 SPARK_CORECORE, U10 AD5248MSOP-10, U11 INA219SOT23-8, U12 INA219SOT23-8, U13 INA219SOT23-8, U14 INA219SOT23-8, U15 INA219SOT23-8, U16 MIC29300D2PAK-3, U17 L7805D2PAK-2, U18 RK7002BSOT23-3, U19 RK7002BSOT23-3, U2 RELAY-SOLIDSTATEPTH, U20 RELAY-SOLIDSTATEPTH, U21 RELAY-SOLIDSTATEPTH, U22 AD5248MSOP-10, U23 CAT4101TO-263, U24 CAT4101TO-263, U25 CAT4101TO-263, U26 INA219SOT23-8, U27 INA219SOT23-8, U28 INA219SOT23-8, U29 DS3231MSOIC-8, U3 CAT4101TO-263, U30 RELAY-SOLIDSTATEPTH, U31 RELAY-SOLIDSTATEPTH, U4 CAT4101TO-263, U5 CAT4101TO-263, U6 CAT4101TO-263, U7 CAT4101TO-263, U8 AD5248MSOP-10, U9 AD5248MSOP-10

Commit message: FishLight_PCB: Fix Spark pin assignments
The Spark Core schematic symbol is a bit misleading.  The RAW pin is
actually VIN, VDDA is the 'clean' 3.3V output from the voltage
regulator, and VDD is actually the 3.3V pin, which could power the Core
if I was using a 3.3V regulator.  Also, all analog pins are PWM pins and
the D0/D1 pins are SDA/SCL.  I also fixed the CAT4101 connections to
connect to actual PWM pins.
Connections:
- removed net D0: U1.D0, U3.PWM, U7.PWM
- removed net D1: U1.D1, U23.PWM, U4.PWM
- new net 3.3A: U1.VDDA
- new net 3.3V: U1.VCC
- new net A4: U1.A4
- new net A5: U1.A5
- net 5V: now also U1.RAW; no longer U1.VCC
- net A0: now also U3.PWM, U7.PWM
- net A1: now also U25.PWM, U5.PWM
- net A2: now also U23.PWM, U4.PWM
- net A3: now also U24.PWM, U6.PWM
- net D2: no longer U25.PWM, U5.PWM
- net D3: no longer U24.PWM, U6.PWM
- net SCL: now also U1.D1; no longer U1.A4
- net SDA: now also U1.D0; no longer U1.A5
Other:
- note added: "PWM"
Changed lines of the file:
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@@
 <text x="103.124" y="77.47" size="1.778" layer="91">ADR: 110</text>
 <text x="103.124" y="57.15" size="1.778" layer="91">ADR: 111</text>
+<text x="17.78" y="160.02" size="1.778" layer="91">PWM</text>
+<text x="17.78" y="154.94" size="1.778" layer="91">PWM</text>
+<text x="17.78" y="149.86" size="1.778" layer="91">PWM</text>
+<text x="17.78" y="144.78" size="1.778" layer="91">PWM</text>
+<text x="17.78" y="139.7" size="1.778" layer="91">PWM</text>
+<text x="17.78" y="134.62" size="1.778" layer="91">PWM</text>
+<text x="17.78" y="129.54" size="1.778" layer="91">PWM</text>
+<text x="17.78" y="124.46" size="1.778" layer="91">PWM</text>
 </plain>
 <instances>
@@
 <net name="SDA" class="0">
 <segment>
-<wire x1="7.62" y1="149.86" x2="2.54" y2="149.86" width="0.1524" layer="91"/>
-<label x="2.54" y="149.86" size="1.778" layer="91"/>
-<pinref part="U1" gate="G$1" pin="A5"/>
-</segment>
-<segment>
 <wire x1="231.14" y1="45.72" x2="233.68" y2="45.72" width="0.1524" layer="91"/>
 <label x="231.14" y="45.72" size="1.778" layer="95"/>
@@
 <label x="114.3" y="71.12" size="1.778" layer="95"/>
 </segment>
+<segment>
+<pinref part="U1" gate="G$1" pin="D0"/>
+<wire x1="43.18" y1="124.46" x2="48.26" y2="124.46" width="0.2032" layer="91"/>
+<label x="43.18" y="124.46" size="1.778" layer="95"/>
+</segment>
 </net>
 <net name="SCL" class="0">
-<segment>
-<wire x1="7.62" y1="144.78" x2="2.54" y2="144.78" width="0.1524" layer="91"/>
-<label x="2.54" y="144.78" size="1.778" layer="91"/>
-<pinref part="U1" gate="G$1" pin="A4"/>
-</segment>
 <segment>
 <wire x1="231.14" y1="48.26" x2="233.68" y2="48.26" width="0.1524" layer="91"/>
@@
 <wire x1="114.3" y1="50.8" x2="119.38" y2="50.8" width="0.2032" layer="91"/>
 <label x="114.3" y="50.8" size="1.778" layer="95"/>
+</segment>
+<segment>
+<pinref part="U1" gate="G$1" pin="D1"/>
+<wire x1="43.18" y1="129.54" x2="48.26" y2="129.54" width="0.2032" layer="91"/>
+<label x="43.18" y="129.54" size="1.778" layer="95"/>
 </segment>
 </net>
@@
 <net name="5V" class="0">
 <segment>
-<wire x1="48.26" y1="180.34" x2="43.18" y2="180.34" width="0.1524" layer="91"/>
-<label x="43.18" y="180.34" size="1.778" layer="91"/>
-<pinref part="U1" gate="G$1" pin="VCC"/>
-</segment>
-<segment>
 <wire x1="205.74" y1="45.72" x2="210.82" y2="45.72" width="0.1524" layer="91"/>
 <label x="205.74" y="45.72" size="1.778" layer="95"/>
@@
 <label x="205.74" y="55.88" size="1.778" layer="95"/>
 </segment>
+<segment>
+<pinref part="U1" gate="G$1" pin="RAW"/>
+<wire x1="7.62" y1="180.34" x2="2.54" y2="180.34" width="0.2032" layer="91"/>
+<label x="2.54" y="180.34" size="1.778" layer="95"/>
+</segment>
 </net>
 <net name="SQW" class="0">
@@
 <pinref part="U1" gate="G$1" pin="A0"/>
 </segment>
+<segment>
+<pinref part="U3" gate="G$1" pin="PWM"/>
+<wire x1="134.62" y1="180.34" x2="129.54" y2="180.34" width="0.2032" layer="91"/>
+<label x="129.54" y="180.34" size="1.778" layer="95"/>
+</segment>
+<segment>
+<pinref part="U7" gate="G$1" pin="PWM"/>
+<wire x1="134.62" y1="149.86" x2="129.54" y2="149.86" width="0.2032" layer="91"/>
+<label x="129.54" y="149.86" size="1.778" layer="95"/>
+</segment>
 </net>
 <net name="A1" class="0">
@@
 <pinref part="U1" gate="G$1" pin="A1"/>
 </segment>
+<segment>
+<pinref part="U5" gate="G$1" pin="PWM"/>
+<wire x1="134.62" y1="165.1" x2="129.54" y2="165.1" width="0.2032" layer="91"/>
+<label x="129.54" y="165.1" size="1.778" layer="95"/>
+</segment>
+<segment>
+<pinref part="U25" gate="G$1" pin="PWM"/>
+<wire x1="134.62" y1="134.62" x2="129.54" y2="134.62" width="0.2032" layer="91"/>
+<label x="129.54" y="134.62" size="1.778" layer="95"/>
+</segment>
 </net>
 <net name="A2" class="0">
@@
 <pinref part="U1" gate="G$1" pin="A2"/>
 </segment>
+<segment>
+<pinref part="U4" gate="G$1" pin="PWM"/>
+<wire x1="167.64" y1="180.34" x2="162.56" y2="180.34" width="0.2032" layer="91"/>
+<label x="162.56" y="180.34" size="1.778" layer="95"/>
+</segment>
+<segment>
+<pinref part="U23" gate="G$1" pin="PWM"/>
+<wire x1="167.64" y1="149.86" x2="162.56" y2="149.86" width="0.2032" layer="91"/>
+<label x="162.56" y="149.86" size="1.778" layer="95"/>
+</segment>
 </net>
 <net name="A3" class="0">
@@
 <label x="2.54" y="139.7" size="1.778" layer="95"/>
 <pinref part="U1" gate="G$1" pin="A3"/>
+</segment>
+<segment>
+<pinref part="U6" gate="G$1" pin="PWM"/>
+<wire x1="167.64" y1="165.1" x2="162.56" y2="165.1" width="0.2032" layer="91"/>
+<label x="162.56" y="165.1" size="1.778" layer="95"/>
+</segment>
+<segment>
+<pinref part="U24" gate="G$1" pin="PWM"/>
+<wire x1="167.64" y1="134.62" x2="162.56" y2="134.62" width="0.2032" layer="91"/>
+<label x="162.56" y="134.62" size="1.778" layer="95"/>
 </segment>
 </net>
@@
 <pinref part="U1" gate="G$1" pin="D3"/>
 </segment>
-<segment>
-<pinref part="U6" gate="G$1" pin="PWM"/>
-<wire x1="167.64" y1="165.1" x2="162.56" y2="165.1" width="0.2032" layer="91"/>
-<label x="162.56" y="165.1" size="1.778" layer="95"/>
-</segment>
-<segment>
-<pinref part="U24" gate="G$1" pin="PWM"/>
-<wire x1="167.64" y1="134.62" x2="162.56" y2="134.62" width="0.2032" layer="91"/>
-<label x="162.56" y="134.62" size="1.778" layer="95"/>
-</segment>
 </net>
 <net name="D2" class="0">
@@
 <label x="43.18" y="134.62" size="1.778" layer="95"/>
 <pinref part="U1" gate="G$1" pin="D2"/>
-</segment>
-<segment>
-<pinref part="U5" gate="G$1" pin="PWM"/>
-<wire x1="134.62" y1="165.1" x2="129.54" y2="165.1" width="0.2032" layer="91"/>
-<label x="129.54" y="165.1" size="1.778" layer="95"/>
-</segment>
-<segment>
-<pinref part="U25" gate="G$1" pin="PWM"/>
-<wire x1="134.62" y1="134.62" x2="129.54" y2="134.62" width="0.2032" layer="91"/>
-<label x="129.54" y="134.62" size="1.778" layer="95"/>
 </segment>
 </net>
@@
 </segment>
 </net>
-<net name="D1" class="0">
-<segment>
-<pinref part="U1" gate="G$1" pin="D1"/>
-<wire x1="43.18" y1="129.54" x2="48.26" y2="129.54" width="0.2032" layer="91"/>
-<label x="43.18" y="129.54" size="1.778" layer="95"/>
-</segment>
-<segment>
-<pinref part="U4" gate="G$1" pin="PWM"/>
-<wire x1="167.64" y1="180.34" x2="162.56" y2="180.34" width="0.2032" layer="91"/>
-<label x="162.56" y="180.34" size="1.778" layer="95"/>
-</segment>
-<segment>
-<pinref part="U23" gate="G$1" pin="PWM"/>
-<wire x1="167.64" y1="149.86" x2="162.56" y2="149.86" width="0.2032" layer="91"/>
-<label x="162.56" y="149.86" size="1.778" layer="95"/>
-</segment>
-</net>
 <net name="A7" class="0">
 <segment>
@@
 <wire x1="7.62" y1="154.94" x2="2.54" y2="154.94" width="0.2032" layer="91"/>
 <label x="2.54" y="154.94" size="1.778" layer="95"/>
-</segment>
-</net>
-<net name="D0" class="0">
-<segment>
-<pinref part="U1" gate="G$1" pin="D0"/>
-<wire x1="43.18" y1="124.46" x2="48.26" y2="124.46" width="0.2032" layer="91"/>
-<label x="43.18" y="124.46" size="1.778" layer="95"/>
-</segment>
-<segment>
-<pinref part="U3" gate="G$1" pin="PWM"/>
-<wire x1="134.62" y1="180.34" x2="129.54" y2="180.34" width="0.2032" layer="91"/>
-<label x="129.54" y="180.34" size="1.778" layer="95"/>
-</segment>
-<segment>
-<pinref part="U7" gate="G$1" pin="PWM"/>
-<wire x1="134.62" y1="149.86" x2="129.54" y2="149.86" width="0.2032" layer="91"/>
-<label x="129.54" y="149.86" size="1.778" layer="95"/>
 </segment>
 </net>
@@
 </segment>
 </net>
+<net name="A5" class="0">
+<segment>
+<pinref part="U1" gate="G$1" pin="A5"/>
+<wire x1="7.62" y1="149.86" x2="2.54" y2="149.86" width="0.2032" layer="91"/>
+<label x="2.54" y="149.86" size="1.778" layer="95"/>
+</segment>
+</net>
+<net name="A4" class="0">
+<segment>
+<pinref part="U1" gate="G$1" pin="A4"/>
+<wire x1="7.62" y1="144.78" x2="2.54" y2="144.78" width="0.2032" layer="91"/>
+<label x="2.54" y="144.78" size="1.778" layer="95"/>
+</segment>
+</net>
+<net name="3.3V" class="0">
+<segment>
+<pinref part="U1" gate="G$1" pin="VCC"/>
+<wire x1="43.18" y1="180.34" x2="48.26" y2="180.34" width="0.2032" layer="91"/>
+<label x="43.18" y="180.34" size="1.778" layer="95"/>
+</segment>
+</net>
+<net name="3.3A" class="0">
+<segment>
+<pinref part="U1" gate="G$1" pin="VDDA"/>
+<wire x1="43.18" y1="170.18" x2="48.26" y2="170.18" width="0.2032" layer="91"/>
+<label x="43.18" y="170.18" size="1.778" layer="95"/>
+</segment>
+</net>

Commit message: FishLight_PCB: Started work on 12V devices
The 12V devices require the ability to turn them on and off but also to
hold them on or off without constant need of the Spark Core to supply a
transistor.  I am going to use a MUX with a D Flip-Flop and a transistor
to hold the devices High or Low and then go and do other things while
the FF holds their state.  I have placed the MUXes, the beginnings of
the FF circuit, and the terminals.  I have also connected the Spark
outputs D2 - D5 to the MUX S inputs.  I also changed the TMP sensors to
D6.
Parts:
- added JP28, JP29, JP30, JP31, JP32: M023.5MM, SparkFun-Connectors:M023.5MM
- added LED1: (no value), SparkFun-LED:LED0603
- added R16: (no value), SparkFun-Resistors:RESISTOR0603
- added U$1, U$2: CD74HC4067SSOP24, Mikes-Stuff:CD74HC4067SSOP24
- added U$3: NC7SZ373, Mikes-Stuff:NC7SZ373
- added U$4: RK7002BSOT23-3, Mikes-Stuff:RK7002BSOT23-3
Connections:
- new net DCOM: U$1.COM
- new net ECOM: U$2.COM
- new net N$20: U$1.I8
- new net N$22: U$1.I9
- new net N$24: U$1.I10
- new net N$26: U$1.I11
- new net N$28: U$1.I12
- new net N$30: U$1.I13
- new net N$31: U$1.I14
- new net N$32: U$1.I15
- new net N$49: U$1.I7
- new net N$50: U$1.I6
- new net N$51: U$1.I5
- new net N$52: U$1.I4
- new net N$53: U$1.I3
- new net N$54: U$1.I2
- new net N$55: U$1.I1
- new net N$56: U$1.I0
- new net N$72: JP28.1, U20.T1
- new net N$73: JP28.2, U20.T2
- new net N$74: JP29.1, U21.T1
- new net N$75: JP29.2, U21.T2
- new net N$76: JP30.1, U2.T1
- new net N$77: JP30.2, U2.T2
- new net N$78: JP31.1, U30.T1
- new net N$79: JP31.2, U30.T2
- new net N$80: JP32.1, U31.T1
- new net N$81: JP32.2, U31.T2
- net 5V: now also U$1.VCC
- net D2: now also U$1.S0
- net D3: now also U$1.S1
- net D4: now also U$1.S2
- net D5: now also U$1.S3; no longer JP1.2, JP2.2, JP3.2, R4.1
- net D6: now also JP1.2, JP2.2, JP3.2, R4.1
- net GND: now also U$1.E_, U$1.GND
Other:
- note added: "12V Devs"
- note added: "AC Devs"
- note added: "D input to Flip Flop"
- note added: "E input to Flip Flop"
- moved on the sheet: JP17, JP19, JP21, JP22, JP23, JP24, JP25, JP26, JP27, U2, U20, U21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

Commit message: FishLight_PCB: Update D-Latch symbol
The D-Latch symbol was really big.  I was able to make it a bit smaller
so that I could fit a bunch of these circuits onto the schematic.
Parts:
- U$3: value NC7SZ373 -> NC7SZ373TSSOP-6; device Mikes-Stuff:NC7SZ373 -> Mikes-Stuff:NC7SZ373TSSOP-6
Connections:
- new net N$37: U$2.I8
- new net N$38: U$2.I9
- new net N$39: U$2.I10
- new net N$40: U$2.I11
- new net N$41: U$2.I12
- new net N$42: U$2.I13
- new net N$43: U$2.I14
- new net N$44: U$2.I15
- new net N$61: U$2.I7
- new net N$62: U$2.I6
- new net N$63: U$2.I5
- new net N$64: U$2.I4
- new net N$65: U$2.I3
- new net N$66: U$2.I2
- new net N$67: U$2.I1
- new net N$68: U$2.I0
- net 5V: now also U$2.VCC
- net D2: now also U$2.S0
- net D3: now also U$2.S1
- net D4: now also U$2.S2
- net D5: now also U$2.S3
- net GND: now also U$2.E_, U$2.GND
Other:
- note added: "LE input to Flip Flop"
- note removed: "E input to Flip Flop"
- moved on the sheet: U$1, U$2, U$3

Commit message: FishLight_PCB: Created 12V circuits and fixed fans
Fixed up the fan circuits to be a bit better and to to take less space.
Also created a circuit with the D-Latch, Mosfet, MUX, and LED for the
12V devices.  Created 8 instances so far.  Will probably get rid of a
few of the AC switches and replace with 12V devices.
Parts:
- added LED2, LED3, LED4, LED5, LED6, LED7, LED8: (no value), SparkFun-LED:LED0603
- added R17, R20, R23, R26, R29, R32, R35, R38: 330, SparkFun-Resistors:RESISTOR0603
- added R18, R21, R24, R27, R30, R33, R36, R39: 10K, SparkFun-Resistors:RESISTOR0603-RES
- added R19, R22, R25, R28, R31, R34, R37: (no value), SparkFun-Resistors:RESISTOR0603
- added U$10, U$12, U$14, U$16, U$18, U$20, U$8: RK7002BSOT23-3, Mikes-Stuff:RK7002BSOT23-3
- added U$11, U$13, U$15, U$17, U$19, U$5, U$6, U$7, U$9: NC7SZ373TSSOP-6, Mikes-Stuff:NC7SZ373TSSOP-6
- JP17, JP19, JP21, JP22, JP23, JP24, JP25, JP26, JP27: value M023.5MM -> M022.54MM_SCREWTERM; device SparkFun-Connectors:M023.5MM -> Mikes-Stuff:M022.54MM_SCREWTERM
Connections:
- net N$20 renamed DL8
- net N$22 renamed DL9
- net N$24 renamed DL10
- net N$26 renamed DL11
- net N$28 renamed DL12
- net N$30 renamed DL13
- net N$31 renamed DL14
- net N$32 renamed DL15
- net N$37 renamed LE8
- net N$38 renamed LE9
- net N$39 renamed LE10
- net N$40 renamed LE11
- net N$41 renamed LE12
- net N$42 renamed LE13
- net N$43 renamed LE14
- net N$44 renamed LE15
- net N$49 renamed DL7
- net N$50 renamed DL6
- net N$51 renamed DL5
- net N$52 renamed DL4
- net N$53 renamed DL3
- net N$54 renamed DL2
- net N$61 renamed LE7
- net N$62 renamed LE6
- net N$63 renamed LE5
- net N$64 renamed LE4
- net N$65 renamed LE3
- net N$66 renamed LE2
- new net DL0: U$1.I0, U$5.D
- new net DL1: U$1.I1, U$6.D
- new net LE0: U$2.I0, U$5.LE
- new net LE1: U$2.I1, U$6.LE
- new net N$14: R16.2, R17.1, U$4.G
- new net N$20: R19.2, R20.1, U$8.G
- new net N$22: R20.2, R21.2, U$7.Q
- new net N$24: LED2.C, R19.1
- new net N$26: U$7.GND
- new net N$28: R22.2, R23.1, U$10.G
- new net N$30: R23.2, R24.2, U$9.Q
- new net N$31: LED3.C, R22.1
- new net N$32: U$9.GND
- new net N$33: R17.2, R18.2, U$3.Q
- new net N$34: R25.2, R26.1, U$12.G
- new net N$35: R28.2, R29.1, U$14.G
- new net N$36: R26.2, R27.2, U$11.Q
- new net N$37: LED4.C, R25.1
- new net N$38: U$11.GND
- new net N$39: R29.2, R30.2, U$13.Q
- new net N$40: LED5.C, R28.1
- new net N$41: U$13.GND
- new net N$42: R31.2, R32.1, U$16.G
- new net N$43: R32.2, R33.2, U$15.Q
- new net N$44: LED6.C, R31.1
- new net N$45: LED1.C, R16.1
- new net N$46: U$15.GND
- new net N$47: R34.2, R35.1, U$18.G
- new net N$48: U$3.GND
- new net N$49: R35.2, R36.2, U$17.Q
- new net N$50: LED7.C, R34.1
- new net N$51: U$17.GND
- new net N$52: R37.2, R38.1, U$20.G
- new net N$53: R38.2, R39.2, U$19.Q
- new net N$54: LED8.C, R37.1
- new net N$57: U$3.D
- new net N$58: U$4.D
- new net N$59: U$13.LE
- new net N$60: U$13.D
- new net N$61: U$15.LE
- new net N$62: U$15.D
- new net N$63: U$8.D
- new net N$64: U$7.LE
- new net N$65: U$7.D
- new net N$66: U$9.LE
- new net N$69: U$17.LE
- new net N$70: U$17.D
- new net N$71: U$18.D
- new net N$82: U$16.D
- new net N$83: U$14.D
- new net N$84: U$20.D
- new net N$85: U$12.D
- new net N$86: U$19.LE
- new net N$87: U$19.D
- new net N$88: U$11.LE
- new net N$89: U$11.D
- net 5V: now also LED1.A, LED2.A, LED3.A, LED4.A, LED5.A, LED6.A, LED7.A, LED8.A, U$11.VCC, U$13.VCC, U$15.VCC, U$17.VCC, U$19.VCC, U$3.VCC, U$5.VCC, U$6.VCC, U$7.VCC, U$9.VCC
- net FAN1: now also U$5.Q
- net FAN2: now also U$6.Q
- net GND: now also R18.1, R21.1, R24.1, R27.1, R30.1, R33.1, R36.1, R39.1, U$10.S, U$11./OE, U$12.S, U$13./OE, U$14.S, U$15./OE, U$16.S, U$17./OE, U$18.S, U$19./OE, U$20.S, U$3./OE, U$4.S, U$5./OE, U$5.GND, U$6./OE, U$6.GND, U$7./OE, U$8.S, U$9./OE
- net N$55: now also U$19.GND; no longer U$1.I1
- net N$56: now also U$3.LE; no longer U$1.I0
- net N$67: now also U$9.D; no longer U$2.I1
- net N$68: now also U$10.D; no longer U$2.I0
Other:
- note added: "Fans"
- note added: "LE input to Flip Flop (clock)"
- note removed: "LE input to Flip Flop"
- moved on the sheet: JP4, JP5, LED1, R11, R12, R16, R3, R5, U$3, U$4, U18, U19

Commit message: FishLight_PCB: Finish 12V and AC devices
The AC and 12V devices control circuitry is finished.  Now to just place
the parts and start laying them out.  Also made sure to include enough
decoupling caps for all 17 new parts.
Parts:
- removed JP29: M023.5MM, SparkFun-Connectors:M023.5MM
- removed U2, U20, U21: RELAY-SOLIDSTATEPTH, SparkFun-Electromechanical:RELAY-SOLIDSTATEPTH
- added C26, C27, C28, C29, C30, C31, C32, C33, C34, C35, C36, C37, C38, C39, C40, C41, C42: 0.1uF, SparkFun-Capacitors:0.1UF-25V(+80/-20%)(0603)
- added LED10, LED11, LED12, LED13, LED9: (no value), SparkFun-LED:LED0603
- added R40, R43, R46, R49, R52: 150, SparkFun-Resistors:RESISTOR0603
- added R41, R44, R47, R50, R53: 330, SparkFun-Resistors:RESISTOR0603
- added R42, R45, R48, R51, R54, R55, R56, R57: 10K, SparkFun-Resistors:RESISTOR0603-RES
- added U$21, U$23, U$25, U$27, U$29: NC7SZ373TSSOP-6, Mikes-Stuff:NC7SZ373TSSOP-6
- added U$22, U$24, U$26, U$28, U$30: RK7002BSOT23-3, Mikes-Stuff:RK7002BSOT23-3
- added U32: RELAY-SOLIDSTATEPTH, SparkFun-Electromechanical:RELAY-SOLIDSTATEPTH
- JP28: value M023.5MM -> M022.54MM_SCREWTERM; device SparkFun-Connectors:M023.5MM -> Mikes-Stuff:M022.54MM_SCREWTERM
- R16, R19, R22, R25, R28, R31, R34, R37: value (none) -> 150
Connections:
- removed net N$17: JP21.1, JP26.1
- removed net N$21: JP24.1, JP27.1
- removed net N$29: JP25.1
- removed net N$56: U$3.LE
- removed net N$57: U$3.D
- removed net N$58: U$4.D
- removed net N$59: U$13.LE
- removed net N$6: JP19.1
- removed net N$60: U$13.D
- removed net N$61: U$15.LE
- removed net N$62: U$15.D
- removed net N$63: U$8.D
- removed net N$64: U$7.LE
- removed net N$65: U$7.D
- removed net N$66: U$9.LE
- removed net N$67: U$9.D
- removed net N$68: U$10.D
- removed net N$69: U$17.LE
- removed net N$70: U$17.D
- removed net N$71: U$18.D
- removed net N$82: U$16.D
- removed net N$83: U$14.D
- removed net N$84: U$20.D
- removed net N$85: U$12.D
- removed net N$86: U$19.LE
- removed net N$87: U$19.D
- removed net N$88: U$11.LE
- removed net N$89: U$11.D
- new net DC10: JP22.2, U$16.D
- new net DC11: JP17.2, U$14.D
- new net DC12: U$26.D, U30.-
- new net DC13: U$28.D, U31.-
- new net DC14: U$30.D, U32.-
- new net DC2: JP19.2, U$4.D
- new net DC3: JP21.2, U$8.D
- new net DC4: JP24.2, U$10.D
- new net DC5: JP25.2, U$12.D
- new net DC6: JP27.2, U$22.D
- new net DC7: JP28.2, U$24.D
- new net DC8: JP26.2, U$20.D
- new net DC9: JP23.2, U$18.D
- new net N$100: R46.2, R47.1, U$26.G
- new net N$102: R47.2, R48.2, U$25.Q
- new net N$103: LED11.C, R46.1
- new net N$104: U$25.GND
- new net N$105: R49.2, R50.1, U$28.G
- new net N$106: R50.2, R51.2, U$27.Q
- new net N$107: LED12.C, R49.1
- new net N$108: U$27.GND
- new net N$109: R52.2, R53.1, U$30.G
- new net N$110: R53.2, R54.2, U$29.Q
- new net N$111: LED13.C, R52.1
- new net N$112: U$29.GND
- new net N$90: R43.2, R44.1, U$24.G
- new net N$91: R44.2, R45.2, U$23.Q
- new net N$92: LED10.C, R43.1
- new net N$93: U$23.GND
- net 12V: now also JP17.1, JP19.1, JP21.1, JP22.1, JP23.1, JP24.1, JP25.1, JP26.1, JP27.1, JP28.1
- net 5V: now also C26.1, C27.1, C28.1, C29.1, C30.1, C31.1, C32.1, C33.1, C34.1, C35.1, C36.1, C37.1, C38.1, C39.1, C40.1, C41.1, C42.1, LED10.A, LED11.A, LED12.A, LED13.A, LED9.A, R55.1, R56.1, R57.1, U$21.VCC, U$23.VCC, U$25.VCC, U$27.VCC, U$29.VCC
- net DL10: now also U$15.D
- net DL11: now also U$13.D
- net DL12: now also U$25.D
- net DL13: now also U$27.D
- net DL14: now also U$29.D
- net DL2: now also U$3.D
- net DL3: now also U$7.D
- net DL4: now also U$9.D
- net DL5: now also U$11.D
- net DL6: now also U$21.D
- net DL7: now also U$23.D
- net DL8: now also U$19.D
- net DL9: now also U$17.D
- net GND: now also C26.2, C27.2, C28.2, C29.2, C30.2, C31.2, C32.2, C33.2, C34.2, C35.2, C36.2, C37.2, C38.2, C39.2, C40.2, C41.2, C42.2, R42.1, R45.1, R48.1, R51.1, R54.1, U$21./OE, U$22.S, U$23./OE, U$24.S, U$25./OE, U$26.S, U$27./OE, U$28.S, U$29./OE, U$30.S; no longer JP17.2, JP19.2, JP21.2, JP22.2, JP23.2, JP24.2, JP25.2, JP26.2, JP27.2
- net LE10: now also U$15.LE
- net LE11: now also U$13.LE
- net LE12: now also U$25.LE
- net LE13: now also U$27.LE
- net LE14: now also U$29.LE
- net LE2: now also U$3.LE
- net LE3: now also U$7.LE
- net LE4: now also U$9.LE
- net LE5: now also U$11.LE
- net LE6: now also U$21.LE
- net LE7: now also U$23.LE
- net LE8: now also U$19.LE
- net LE9: now also U$17.LE
- net N$23: now also R55.2, U30.+; no longer JP23.1
- net N$25: now also R56.2, U31.+; no longer JP22.1
- net N$27: now also R57.2, U32.+; no longer JP17.1
- net N$72: now also R40.2, R41.1, U$22.G; no longer JP28.1, U20.T1
- net N$73: now also R41.2, R42.2, U$21.Q; no longer JP28.2, U20.T2
- net N$74: now also LED9.C, R40.1; no longer JP29.1, U21.T1
- net N$75: now also U$21.GND; no longer JP29.2, U21.T2
- net N$76: now also U32.T1; no longer U2.T1
- net N$77: now also U32.T2; no longer U2.T2
Other:
- note added: "LED: 2.2V, 20mA"
- moved on the sheet: JP17, JP19, JP21, JP22, JP23, JP24, JP25, JP26, JP27, JP28, JP30, JP31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
