File: FishLight-v01.sch (EAGLE design)
At the start: 209 parts, among them U1 SPARK_CORECORE, U10 AD5248MSOP-10, U11 INA219SOT23-8, U12 INA219SOT23-8, U13 INA219SOT23-8, U14 INA219SOT23-8, U15 INA219SOT23-8, U16 MIC29300D2PAK-3, U17 L7805D2PAK-2, U18 RK7002BSOT23-3, U19 RK7002BSOT23-3, U22 AD5248MSOP-10, U23 CAT4101TO-263, U24 CAT4101TO-263, U25 CAT4101TO-263, U26 INA219SOT23-8, U27 INA219SOT23-8, U28 INA219SOT23-8, U29 DS3231MSOIC-8, U3 CAT4101TO-263, U30 RELAY-SOLIDSTATEPTH, U31 RELAY-SOLIDSTATEPTH, U32 RELAY-SOLIDSTATEPTH, U4 CAT4101TO-263, U5 CAT4101TO-263, U6 CAT4101TO-263, U7 CAT4101TO-263, U8 AD5248MSOP-10, U9 AD5248MSOP-10

Commit message: FishLight_PCB: Placed 12V power circuits
Got all of the 12V power circuitry placed in their general locations.
Need to space them out a bit so that I can actually get in there to
solder them and not violate the DRC.  I may need to increase the board
size a bit to fit the AC SSRs
Parts:
- removed U$1, U$2: CD74HC4067SSOP24, Mikes-Stuff:CD74HC4067SSOP24
- added U2: DS3231MSOIC-8, Mikes-Stuff:DS3231MSOIC-8
- added U33: RELAY-SOLIDSTATEPTH, SparkFun-Electromechanical:RELAY-SOLIDSTATEPTH
- U29: value DS3231MSOIC-8 -> CD74HC4067SSOP24; device Mikes-Stuff:DS3231MSOIC-8 -> Mikes-Stuff:CD74HC4067SSOP24
- U30: value RELAY-SOLIDSTATEPTH -> CD74HC4067SSOP24; device SparkFun-Electromechanical:RELAY-SOLIDSTATEPTH -> Mikes-Stuff:CD74HC4067SSOP24
- renumbered U$10 to Q3, U$11 to U37, U$12 to Q4, U$13 to U43, U$14 to Q10, U$15 to U42, U$16 to Q9, U$17 to U41, U$18 to Q8, U$19 to U40, U$20 to Q7, U$21 to U38, U$22 to Q5, U$23 to U39, U$24 to Q6, U$25 to U48, U$26 to Q11, U$27 to U47, U$28 to Q12, U$29 to U46, U$3 to U34, U$30 to Q13, U$4 to Q1, U$5 to U44, U$6 to U45, U$7 to U35, U$8 to Q2, U$9 to U36, U18 to Q14, U19 to Q15
Connections:
- net 5V: now also U2.VCC, U30.VCC; no longer U$1.VCC, U$2.VCC
- net D2: now also U29.S0, U30.S0; no longer U$1.S0, U$2.S0
- net D3: now also U29.S1, U30.S1; no longer U$1.S1, U$2.S1
- net D4: now also U29.S2, U30.S2; no longer U$1.S2, U$2.S2
- net D5: now also U29.S3, U30.S3; no longer U$1.S3, U$2.S3
- net DC12: now also U31.-; no longer U30.-
- net DC13: now also U32.-; no longer U31.-
- net DC14: now also U33.-; no longer U32.-
- net DCOM: now also U30.COM; no longer U$1.COM
- net DL0: now also U30.I0; no longer U$1.I0
- net DL1: now also U30.I1; no longer U$1.I1
- net DL10: now also U30.I10; no longer U$1.I10
- net DL11: now also U30.I11; no longer U$1.I11
- net DL12: now also U30.I12; no longer U$1.I12
- net DL13: now also U30.I13; no longer U$1.I13
- net DL14: now also U30.I14; no longer U$1.I14
- net DL15: now also U30.I15; no longer U$1.I15
- net DL2: now also U30.I2; no longer U$1.I2
- net DL3: now also U30.I3; no longer U$1.I3
- net DL4: now also U30.I4; no longer U$1.I4
- net DL5: now also U30.I5; no longer U$1.I5
- net DL6: now also U30.I6; no longer U$1.I6
- net DL7: now also U30.I7; no longer U$1.I7
- net DL8: now also U30.I8; no longer U$1.I8
- net DL9: now also U30.I9; no longer U$1.I9
- net ECOM: now also U29.COM; no longer U$2.COM
- net GND: now also U2.GND, U29.E_, U30.E_, U30.GND; no longer U$1.E_, U$1.GND, U$2.E_, U$2.GND
- net LE0: now also U29.I0; no longer U$2.I0
- net LE1: now also U29.I1; no longer U$2.I1
- net LE10: now also U29.I10; no longer U$2.I10
- net LE11: now also U29.I11; no longer U$2.I11
- net LE12: now also U29.I12; no longer U$2.I12
- net LE13: now also U29.I13; no longer U$2.I13
- net LE14: now also U29.I14; no longer U$2.I14
- net LE15: now also U29.I15; no longer U$2.I15
- net LE2: now also U29.I2; no longer U$2.I2
- net LE3: now also U29.I3; no longer U$2.I3
- net LE4: now also U29.I4; no longer U$2.I4
- net LE5: now also U29.I5; no longer U$2.I5
- net LE6: now also U29.I6; no longer U$2.I6
- net LE7: now also U29.I7; no longer U$2.I7
- net LE8: now also U29.I8; no longer U$2.I8
- net LE9: now also U29.I9; no longer U$2.I9
- net N$23: now also U31.+; no longer U30.+
- net N$25: now also U32.+; no longer U31.+
- net N$27: now also U33.+; no longer U32.+
- net N$3: now also U2.VBAT; no longer U29.VBAT
- net N$76: now also U33.T1; no longer U32.T1
- net N$77: now also U33.T2; no longer U32.T2
- net N$78: now also U31.T1; no longer U30.T1
- net N$79: now also U31.T2; no longer U30.T2
- net N$80: now also U32.T1; no longer U31.T1
- net N$81: now also U32.T2; no longer U31.T2
- net SCL: now also U2.SCL; no longer U29.SCL
- net SDA: now also U2.SDA; no longer U29.SDA
- net SQW: now also U2.SQW; no longer U29.SQW
Other:
- moved on the sheet: U31, U32

Commit message: FishLight_PCB: Rearranged some parts
Rearranged the CAT4101s to make more room.  Also changed their screw
terminal assignments to limit the number of crossings.  This will have
to be resolved in software now because the screw terminal assignments
are all screwed around.  Also changed around the Spark to make more room
for the AC SSRs.  These are now placed on the board.  Also moved around
the 12V devices screw terminals and circuitry to limit MUX crossings.
This is going to be super difficult to route and may need to reduce the
number of 12V devices.
Connections:
- net LED1: now also JP20.3; no longer JP12.1
- net LED2: now also JP12.3; no longer JP12.2
- net LED3: now also JP11.1; no longer JP12.3
- net LED4: now also JP11.2; no longer JP11.1
- net LED5: now also JP12.2; no longer JP11.2
- net LED8: now also JP12.1; no longer JP20.3
- net LG1: now also JP16.1; no longer JP9.3
- net LG2: now also JP9.1; no longer JP9.2
- net LG3: now also JP10.3; no longer JP9.1
- net LG4: now also JP10.2; no longer JP10.3
- net LG5: now also JP9.2; no longer JP10.2
- net LG8: now also JP9.3; no longer JP16.1
Changed lines of the file:
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@@
 <net name="LED1" class="0">
-<segment>
-<wire x1="218.44" y1="180.34" x2="213.36" y2="180.34" width="0.2032" layer="91"/>
-<label x="213.36" y="180.34" size="1.778" layer="95"/>
-<pinref part="JP12" gate="G$1" pin="1"/>
-</segment>
 <segment>
 <pinref part="U11" gate="G$1" pin="V-"/>
@@
 <label x="127" y="111.76" size="1.778" layer="95"/>
 </segment>
+<segment>
+<pinref part="JP20" gate="G$1" pin="3"/>
+<wire x1="218.44" y1="149.86" x2="213.36" y2="149.86" width="0.2032" layer="91"/>
+<label x="213.36" y="149.86" size="1.778" layer="95"/>
+</segment>
 </net>
 <net name="LED2" class="0">
-<segment>
-<wire x1="218.44" y1="177.8" x2="213.36" y2="177.8" width="0.2032" layer="91"/>
-<label x="213.36" y="177.8" size="1.778" layer="95"/>
-<pinref part="JP12" gate="G$1" pin="2"/>
-</segment>
 <segment>
 <pinref part="U12" gate="G$1" pin="V-"/>
@@
 <label x="127" y="91.44" size="1.778" layer="95"/>
 </segment>
-</net>
-<net name="LED3" class="0">
-<segment>
+<segment>
+<pinref part="JP12" gate="G$1" pin="3"/>
 <wire x1="218.44" y1="175.26" x2="213.36" y2="175.26" width="0.2032" layer="91"/>
 <label x="213.36" y="175.26" size="1.778" layer="95"/>
-<pinref part="JP12" gate="G$1" pin="3"/>
-</segment>
+</segment>
+</net>
+<net name="LED3" class="0">
 <segment>
 <pinref part="U13" gate="G$1" pin="V-"/>
@@
 <label x="127" y="71.12" size="1.778" layer="95"/>
 </segment>
+<segment>
+<pinref part="JP11" gate="G$1" pin="1"/>
+<wire x1="218.44" y1="167.64" x2="213.36" y2="167.64" width="0.2032" layer="91"/>
+<label x="213.36" y="167.64" size="1.778" layer="95"/>
+</segment>
 </net>
 <net name="LG4" class="0">
@@
 </segment>
 <segment>
-<wire x1="241.3" y1="167.64" x2="246.38" y2="167.64" width="0.2032" layer="91"/>
-<label x="241.3" y="167.64" size="1.778" layer="95"/>
-<pinref part="JP10" gate="G$1" pin="3"/>
+<pinref part="JP10" gate="G$1" pin="2"/>
+<wire x1="241.3" y1="165.1" x2="246.38" y2="165.1" width="0.2032" layer="91"/>
+<label x="241.3" y="165.1" size="1.778" layer="95"/>
 </segment>
 </net>
@@
 </segment>
 <segment>
-<wire x1="241.3" y1="165.1" x2="246.38" y2="165.1" width="0.2032" layer="91"/>
-<label x="241.3" y="165.1" size="1.778" layer="95"/>
-<pinref part="JP10" gate="G$1" pin="2"/>
+<pinref part="JP9" gate="G$1" pin="2"/>
+<wire x1="241.3" y1="177.8" x2="246.38" y2="177.8" width="0.2032" layer="91"/>
+<label x="241.3" y="177.8" size="1.778" layer="95"/>
 </segment>
 </net>
@@
 <net name="LG1" class="0">
 <segment>
-<wire x1="241.3" y1="180.34" x2="246.38" y2="180.34" width="0.2032" layer="91"/>
-<label x="241.3" y="180.34" size="1.778" layer="95"/>
-<pinref part="JP9" gate="G$1" pin="3"/>
-</segment>
-<segment>
 <pinref part="U3" gate="G$1" pin="LED"/>
 <wire x1="134.62" y1="175.26" x2="129.54" y2="175.26" width="0.2032" layer="91"/>
 <label x="129.54" y="175.26" size="1.778" layer="95"/>
 </segment>
+<segment>
+<pinref part="JP16" gate="G$1" pin="1"/>
+<wire x1="241.3" y1="149.86" x2="246.38" y2="149.86" width="0.2032" layer="91"/>
+<label x="241.3" y="149.86" size="1.778" layer="95"/>
+</segment>
 </net>
 <net name="LG2" class="0">
-<segment>
-<wire x1="241.3" y1="177.8" x2="246.38" y2="177.8" width="0.2032" layer="91"/>
-<label x="241.3" y="177.8" size="1.778" layer="95"/>
-<pinref part="JP9" gate="G$1" pin="2"/>
-</segment>
 <segment>
 <pinref part="U4" gate="G$1" pin="LED"/>
@@
 <label x="162.56" y="175.26" size="1.778" layer="95"/>
 </segment>
-</net>
-<net name="LG3" class="0">
-<segment>
+<segment>
+<pinref part="JP9" gate="G$1" pin="1"/>
 <wire x1="241.3" y1="175.26" x2="246.38" y2="175.26" width="0.2032" layer="91"/>
 <label x="241.3" y="175.26" size="1.778" layer="95"/>
-<pinref part="JP9" gate="G$1" pin="1"/>
-</segment>
+</segment>
+</net>
+<net name="LG3" class="0">
 <segment>
 <pinref part="U5" gate="G$1" pin="LED"/>
@@
 <label x="129.54" y="160.02" size="1.778" layer="95"/>
 </segment>
+<segment>
+<pinref part="JP10" gate="G$1" pin="3"/>
+<wire x1="241.3" y1="167.64" x2="246.38" y2="167.64" width="0.2032" layer="91"/>
+<label x="241.3" y="167.64" size="1.778" layer="95"/>
+</segment>
 </net>
 <net name="LR3" class="0">
@@
 </net>
 <net name="LED4" class="0">
-<segment>
-<wire x1="218.44" y1="167.64" x2="213.36" y2="167.64" width="0.2032" layer="91"/>
-<label x="213.36" y="167.64" size="1.778" layer="95"/>
-<pinref part="JP11" gate="G$1" pin="1"/>
-</segment>
 <segment>
 <pinref part="U14" gate="G$1" pin="V-"/>
@@
 <label x="127" y="50.8" size="1.778" layer="95"/>
 </segment>
-</net>
-<net name="LED5" class="0">
-<segment>
+<segment>
+<pinref part="JP11" gate="G$1" pin="2"/>
 <wire x1="218.44" y1="165.1" x2="213.36" y2="165.1" width="0.2032" layer="91"/>
 <label x="213.36" y="165.1" size="1.778" layer="95"/>
-<pinref part="JP11" gate="G$1" pin="2"/>
-</segment>
+</segment>
+</net>
+<net name="LED5" class="0">
 <segment>
 <pinref part="U15" gate="G$1" pin="V-"/>
@@
 <wire x1="93.98" y1="111.76" x2="88.9" y2="111.76" width="0.2032" layer="91"/>
 <label x="88.9" y="111.76" size="1.778" layer="95"/>
+</segment>
+<segment>
+<pinref part="JP12" gate="G$1" pin="2"/>
+<wire x1="218.44" y1="177.8" x2="213.36" y2="177.8" width="0.2032" layer="91"/>
+<label x="213.36" y="177.8" size="1.778" layer="95"/>
 </segment>
 </net>
@@
 </segment>
 <segment>
-<pinref part="JP20" gate="G$1" pin="3"/>
-<wire x1="218.44" y1="149.86" x2="213.36" y2="149.86" width="0.2032" layer="91"/>
-<label x="213.36" y="149.86" size="1.778" layer="95"/>
+<pinref part="JP12" gate="G$1" pin="1"/>
+<wire x1="218.44" y1="180.34" x2="213.36" y2="180.34" width="0.2032" layer="91"/>
+<label x="213.36" y="180.34" size="1.778" layer="95"/>
 </segment>
 </net>
@@
 </segment>
 <segment>
-<pinref part="JP16" gate="G$1" pin="1"/>
-<wire x1="241.3" y1="149.86" x2="246.38" y2="149.86" width="0.2032" layer="91"/>
-<label x="241.3" y="149.86" size="1.778" layer="95"/>
-</segment>
-</net>
+<pinref part="JP9" gate="G$1" pin="3"/>
+<wire x1="241.3" y1="180.34" x2="246.38" y2="180.34" width="0.2032" layer="91"/>
+<label x="241.3" y="180.34" size="1.778" layer="95"/>
+</segment>
+</net>

Commit message: FishLight_PCB: Add water level sensors
The water level sensors will be used to sense when a water top off is
needed and to ensure that the water reservoirs do not get too low and
potentially burn out my pumps.  Also removed a temp sensor because I
don't think 3 external temp sensors are really necessary.

Water level sensors are from Adafruit: http://www.adafruit.com/products/464
Parts:
- removed JP3: (no value), Mikes-Stuff:M03POLAR
- added JP29, JP33, JP34: M02POLAR, Mikes-Stuff:M02POLAR
- added R58, R59, R60: 560, SparkFun-Resistors:RESISTOR0603-RES
Connections:
- net 5V: now also R58.2, R59.2, R60.2; no longer JP3.3
- net A4: now also JP29.2, R58.1
- net A5: now also JP33.2, R59.1
- net A6: now also JP34.2, R60.1
- net D6: no longer JP3.2
- net GND: now also JP29.1, JP33.1, JP34.1; no longer JP3.1
Other:
- note added: "Pots"
- note added: "RTC"
- note added: "Water Level Sensors"
- moved on the sheet: BAT1, C1, C10, C11, C13, C16, C17, C19, C2, C20, C21, C22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
