File: FishLight-v01.sch (EAGLE design)
At the start: 213 parts, among them Q1 RK7002BSOT23-3, Q10 RK7002BSOT23-3, Q11 RK7002BSOT23-3, Q12 RK7002BSOT23-3, Q13 RK7002BSOT23-3, Q14 RK7002BSOT23-3, Q15 RK7002BSOT23-3, Q2 RK7002BSOT23-3, Q3 RK7002BSOT23-3, Q4 RK7002BSOT23-3, Q5 RK7002BSOT23-3, Q6 RK7002BSOT23-3, Q7 RK7002BSOT23-3, Q8 RK7002BSOT23-3, Q9 RK7002BSOT23-3, U1 SPARK_CORECORE, U10 AD5248MSOP-10, U11 INA219SOT23-8, U12 INA219SOT23-8, U13 INA219SOT23-8, U14 INA219SOT23-8, U15 INA219SOT23-8, U16 MIC29300D2PAK-3, U17 L7805D2PAK-2, U22 AD5248MSOP-10, U23 CAT4101TO-263, U24 CAT4101TO-263, U25 CAT4101TO-263, U26 INA219SOT23-8, U27 INA219SOT23-8, U28 INA219SOT23-8, U29 CD74HC4067SSOP24, U3 CAT4101TO-263, U30 CD74HC4067SSOP24, U31 RELAY-SOLIDSTATEPTH, U32 RELAY-SOLIDSTATEPTH, U33 RELAY-SOLIDSTATEPTH, U34 NC7SZ373TSSOP-6, U35 NC7SZ373TSSOP-6, U36 NC7SZ373TSSOP-6, U37 NC7SZ373TSSOP-6, U38 NC7SZ373TSSOP-6, U39 NC7SZ373TSSOP-6, U4 CAT4101TO-263, U40 NC7SZ373TSSOP-6, U41 NC7SZ373TSSOP-6, U42 NC7SZ373TSSOP-6, U43 NC7SZ373TSSOP-6, U44 NC7SZ373TSSOP-6, U45 NC7SZ373TSSOP-6, U46 NC7SZ373TSSOP-6, U47 NC7SZ373TSSOP-6, U48 NC7SZ373TSSOP-6, U49 DS18B20USOP8, U5 CAT4101TO-263, U6 CAT4101TO-263, U7 CAT4101TO-263, U8 AD5248MSOP-10, U9 AD5248MSOP-10

Commit message: FishLight_PCB: Start moving the MUX signals around
The signals to the MUXes were all crisscrossed and would be nearly
impossible to route.  I got the LE signals all untangled and started in
on the D signals.
Connections:
- net DL15 renamed N$56
- new net N$10: U30.I8
- new net N$11: U30.I9
- new net N$12: U30.I10
- new net N$19: U30.I13
- new net N$21: U30.I14
- new net N$7: U30.I2
- new net N$8: U30.I1
- new net N$9: U30.I0
- net DL0: no longer U30.I0
- net DL1: no longer U30.I1
- net DL10: no longer U30.I10
- net DL12: no longer U30.I12
- net DL13: no longer U30.I13
- net DL14: no longer U30.I14
- net DL2: now also U30.I3; no longer U30.I2
- net DL3: now also U30.I4; no longer U30.I3
- net DL4: now also U30.I5; no longer U30.I4
- net DL5: now also U30.I6; no longer U30.I5
- net DL6: now also U30.I7; no longer U30.I6
- net DL7: now also U30.I12; no longer U30.I7
- net DL8: no longer U30.I8
- net DL9: no longer U30.I9
- net LE10: now also U29.I4; no longer U29.I10
- net LE11: now also U29.I7; no longer U29.I11
- net LE12: now also U29.I9; no longer U29.I12
- net LE13: now also U29.I10; no longer U29.I13
- net LE14: now also U29.I2; no longer U29.I14
- net LE2: now also U29.I8; no longer U29.I2
- net LE3: now also U29.I14; no longer U29.I3
- net LE4: now also U29.I13; no longer U29.I4
- net LE5: now also U29.I12; no longer U29.I5
- net LE6: now also U29.I11; no longer U29.I6
- net LE7: now also U29.I6; no longer U29.I7
- net LE8: now also U29.I5; no longer U29.I8
- net LE9: now also U29.I3; no longer U29.I9

Commit message: FishLight_PCB: Lots and lots of routing
Most of the routing is done now.  Got the MUX signals mostly figured out
but there are still a few that are going to be very tough, like the AC
devices and the fans.  The AC devices still need to be hooked to their
terminals too and this worries me because there isn't much space to
isolate the lines.  I guess the good news is that if it shorts that just
means it gets connected and it wont be controllable from the Spark.  But
this isn't a good thing either.
Parts:
- removed R58, R59, R60: 560, SparkFun-Resistors:RESISTOR0603-RES
Connections:
- net N$8 renamed DL15
- removed net N$10: U30.I8
- removed net N$11: U30.I9
- removed net N$12: U30.I10
- removed net N$19: U30.I13
- removed net N$21: U30.I14
- removed net N$56: U30.I15
- removed net N$7: U30.I2
- removed net N$9: U30.I0
- net 5V: no longer R58.2, R59.2, R60.2
- net A4: no longer R58.1
- net A5: no longer R59.1
- net A6: no longer R60.1
- net DL0: now also U30.I10
- net DL1: now also U30.I9
- net DL10: now also U30.I14
- net DL12: now also U30.I8
- net DL13: now also U30.I2
- net DL14: now also U30.I0
- net DL8: now also U30.I13
- net DL9: now also U30.I15
Other:
- note added: "Note: Add pullups on Spark Core pins in software"
